File: kicad/usb.kicad_sch (KiCad schematic)
At the start: 4 parts, among them J3 USB_C_Receptacle_USB2.0_16P, U2 USBLC6-2SC6

Commit message: A LOT OF STUFF
I almost finished the schematic part of the tutorial
what remains is part choosing and filling the relevant fields for every component
Connections:
- net USB_CONNECTOR-D+ renamed CONNECTOR_USB_D+
- net USB_CONNECTOR_D- renamed CONNECTOR_USB_D-
Other:
- note added: "USB Type-C Receptacle"
- note added: "as per usb type-c specification"
- note removed: "as per usb c specification"
- note removed: "todo: add an LDO based on codemx power consumption calculator (pcc?) analysis"
