File: kicad/mcu_miscellaneous.kicad_sch (KiCad schematic)
At the start: 16 parts, among them J2 Conn_ARM_SWD_TagConnect_TC2030, J4 Conn_01x04_Pin, SW1 SW_Push, SW2 SW_Push, U4 USBLC6-2SC6

Commit message: refactor(schematic): polish the schematic as much as possible - add new Basmala - fix netlist names almost EVERYWHERE, this is to help with net classes, and to help with building a good habit of naming nets properly - add a 100n capacitor to the SWD connector power pin - update many many other things EVERYWHERE
Parts:
- removed C20: 100n, symbol Device:C_Small
- removed J2: Conn_ARM_SWD_TagConnect_TC2030, Connector:Tag-Connect_TC2030-IDC-FP_2x03_P1.27mm_Vertical, symbol Connector:Conn_ARM_SWD_TagConnect_TC2030
- removed J4: Conn_01x04_Pin, symbol Connector:Conn_01x04_Pin
- removed R5, R6: 220R, symbol Device:R
- removed U4: USBLC6-2SC6, Package_TO_SOT_SMD:SOT-23-6, symbol Power_Protection:USBLC6-2SC6
Connections:
- net MCU_NRST renamed NRST_OUT
- net NRST renamed NRST_IN
Other:
- note removed: "For any connector or exposed interface you typically should add ESD protection to make sure when you're messing around with the board you don't accidentally fry your devices. However, phil says that from his experience these ST mcus are pretty resilient, so it's fine for *test boards* to skip them, however he doesn't recommend this for connectors on commercial boards"
- note removed: "RX of the device is TX of the connector"
- note removed: "Tag-Connect SWD Header"
- note removed: "UART Header"
- note removed: "add a small bypass/decoupling capacitor at any connector power pin"
- note removed: "current-limiting resistors"
- moved on the sheet: C16, C17, D1, D3, R1, R2, R7, R9, SW1, SW2
