File: kicad/mcu_crystals.kicad_sch (KiCad schematic)
At the start: 6 parts, among them X1 32MHz, X2 32kHz768

Commit message: everything: select real components, refactor schematic, add a user-led driving circuit, and more
Parts:
- R1, R2: footprint (none) -> Resistor_SMD:R_0402_1005Metric
- X1: Distributor (none) -> LCSC; MPN (none) -> NX2016SA-32MHZ-EXS00A-CS06654; Manufacturer Part Number NX2016SA-32MHZ-EXS00A-CS06654 -> (none)
- X2: Distributor (none) -> LCSC; Distributor Link (none) -> https://www.lcsc.com/product-detail/C891748.html?s_z=s_p_NX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; MPN (none) -> NX2012SA-32.768KHZ-STD-MUB-2; Manufacturer Part Number NX2012SA-32.768KHZ-STD-MUB-2 -> (none)
Changed lines of the file:
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@@
 			)
 		)
-		(property "Footprint" ""
+		(property "Footprint" "Resistor_SMD:R_0402_1005Metric"
 			(at 146.05 80.01 0)
 			(hide yes)
@@
 		(property "Description" "Resistor, small symbol"
 			(at 146.05 80.01 0)
+			(hide yes)
+			(show_name no)
+			(do_not_autoplace no)
+			(effects
+				(font
+					(size 1.27 1.27)
+				)
+			)
+		)
+		(property "Distributor" ""
+			(at 146.05 80.01 90)
 			(hide yes)
 			(show_name no)
@@
 			)
 		)
-		(property "Datasheet" ""
+		(property "Datasheet" "https://www.lcsc.com/datasheet/C891748.pdf?spm=wm.sxq.inf.ggs___wm.fly.bg.0.xh&lcsc_vid=RlRYUFFURFcNVFIDFVMMXgZSRlJeUABSQVNfAwJfQwIxVlNeTldcXlVQRFddVjsOAxUeFF5JWBYZEEoKFBINSQcJGk4eFQsCAgIaSgADAwAHC0slRFBXUFJeQ08GEwkK"
 			(at 156.21 125.73 0)
 			(hide yes)
@@
 			)
 		)
-		(property "Description" "Two pin crystal"
+		(property "Description" "CRYSTAL 32.768kHz SMD"
 			(at 156.21 125.73 0)
 			(hide yes)
@@
 			)
 		)
-		(property "Distributor Link" ""
+		(property "Distributor Link" "https://www.lcsc.com/product-detail/C891748.html?s_z=s_p_NX2012SA-32.768KHZ-STD-MUB-2&spm=wm.fly.bg.0.xh&lcsc_vid=RlRYUFFURFcNVFIDFVMMXgZSRlJeUABSQVNfAwJfQwIxVlNeTldcXlVQRFddVjsOAxUeFF5JWBYZEEoKFBINSQcJGk4eFQsCAgIaSgADAwAHC0slRFBXUFJeQ08GEwkK"
 			(at 156.21 125.73 0)
 			(hide yes)
@@
 			)
 		)
-		(property "Manufacturer Part Number" "NX2012SA-32.768KHZ-STD-MUB-2"
+		(property "Distributor" "LCSC"
+			(at 156.21 125.73 0)
+			(hide yes)
+			(show_name no)
+			(do_not_autoplace no)
+			(effects
+				(font
+					(size 1.27 1.27)
+				)
+			)
+		)
+		(property "MPN" "NX2012SA-32.768KHZ-STD-MUB-2"
 			(at 156.21 125.73 0)
 			(hide yes)
@@
 			)
 		)
-		(property "Datasheet" ""
+		(property "Datasheet" "https://www.lcsc.com/datasheet/C5441424.pdf?spm=wm.sxq.inf.ggs&lcsc_vid=RlRYUFFURFcNVFIDFVMMXgZSRlJeUABSQVNfAwJfQwIxVlNeTldcXlVeQlNWUDtW"
 			(at 156.21 80.01 0)
 			(hide yes)
@@
 			)
 		)
-		(property "Description" "Four pin crystal, GND on pins 2 and 4"
+		(property "Description" "CRYSTAL 32MHz 8pF SMD"
 			(at 156.21 80.01 0)
 			(hide yes)
@@
 			)
 		)
-		(property "Manufacturer Part Number" "NX2016SA-32MHZ-EXS00A-CS06654"
+		(property "Distributor" "LCSC"
+			(at 156.21 80.01 0)
+			(hide yes)
+			(show_name no)
+			(do_not_autoplace no)
+			(effects
+				(font
+					(size 1.27 1.27)
+				)
+			)
+		)
+		(property "MPN" "NX2016SA-32MHZ-EXS00A-CS06654"
 			(at 156.21 80.01 0)
 			(hide yes)
@@
 			)
 		)
-		(property "Manufacturer Part Number" ""
+		(property "Distributor" ""
 			(at 163.83 132.08 0)
 			(hide yes)
@@
 			)
 		)
-		(property "Manufacturer Part Number" ""
+		(property "Distributor" ""
 			(at 148.59 132.08 0)
 			(hide yes)
@@
 			)
 		)
-		(property "Footprint" ""
+		(property "Footprint" "Resistor_SMD:R_0402_1005Metric"
 			(at 143.51 125.73 0)
 			(hide yes)
@@
 			(hide yes)
 			(show_name no)
+			(do_not_autoplace no)
+			(effects
+				(font
+					(size 1.27 1.27)
+				)
+			)
+		)
+		(property "Distributor" ""
+			(at 143.51 125.73 90)
+			(hide yes)
+			(show_name no)

Commit message: fix(footprints and symbols): add missing footprints and symbols
Parts:
- C14, C15: footprint (none) -> Capacitor_SMD:C_0402_1005Metric
- X1: footprint (none) -> Crystal:Crystal_SMD_2016-4Pin_2.0x1.6mm
- X2: footprint (none) -> Crystal:Crystal_SMD_2012-2Pin_2.0x1.2mm
Changed lines of the file:
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@@
 			)
 		)
-		(property "Footprint" ""
+		(property "Footprint" "Crystal:Crystal_SMD_2012-2Pin_2.0x1.2mm"
 			(at 156.21 125.73 0)
 			(hide yes)
@@
 			)
 		)
-		(property "Footprint" ""
+		(property "Footprint" "Crystal:Crystal_SMD_2016-4Pin_2.0x1.6mm"
 			(at 156.21 80.01 0)
 			(hide yes)
@@
 			)
 		)
-		(property "Footprint" ""
+		(property "Footprint" "Capacitor_SMD:C_0402_1005Metric"
 			(at 164.7952 135.89 0)
 			(hide yes)
@@
 			)
 		)
-		(property "Footprint" ""
+		(property "Footprint" "Capacitor_SMD:C_0402_1005Metric"
 			(at 149.5552 135.89 0)
 			(hide yes)
