File: kicad/connectors.kicad_sch (KiCad schematic)
At the start: 0 parts

Commit message: fix(schematic): misc. fixes and stuff - sort all sheets - add the author's name to all sheets and update the date - add 0R resistor to the input of each crystal oscillator - reannotate all symbols - remove todo.md
Other:
- note added: "+3V3_SWD"
- note added: "+5V_USB"
Changed lines of the file:
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@@
 	(paper "A4")
 	(title_block
-		(date "2026-05-27")
+		(date "2026-06-30")
 		(rev "1.0")
+		(comment 3 "Author: Odai J.")
 		(comment 4 "GitHub: https://github.com/odaij/stm32-bt-board")
 	)
@@
 		)
 	)
+	(text "+5V_USB"
+		(exclude_from_sim no)
+		(at 83.82 86.36 0)
+		(effects
+			(font
+				(size 1.27 1.27)
+				(thickness 0.254)
+				(bold yes)
+			)
+			(justify left)
+		)
+	)
+	(text "+3V3_SWD"
+		(exclude_from_sim no)
+		(at 170.18 86.36 0)
+		(effects
+			(font
+				(size 1.27 1.27)
+				(thickness 0.254)
+				(bold yes)
+			)
+			(justify left)
+		)
+	)
+	(polyline
+		(pts
+			(xy 81.28 86.36) (xy 83.82 86.36)
+		)
+		(stroke
+			(width 0)
+			(type default)
+		)
+	)
 	(wire
 		(pts
@@
 	(wire
 		(pts
-			(xy 175.26 86.36) (xy 167.64 86.36)
-		)
-		(stroke
-			(width 0)
-			(type default)
-		)
-	)
-	(wire
-		(pts
-			(xy 167.64 88.9) (xy 175.26 88.9)
+			(xy 175.26 93.98) (xy 167.64 93.98)
+		)
+		(stroke
+			(width 0)
+			(type default)
+		)
+	)
+	(polyline
+		(pts
+			(xy 167.64 86.36) (xy 170.18 86.36)
+		)
+		(stroke
+			(width 0)
+			(type default)
+		)
+	)
+	(wire
+		(pts
+			(xy 167.64 96.52) (xy 175.26 96.52)
 		)
 		(stroke
@@
 	(hierarchical_label "SWNRST"
 		(shape output)
-		(at 175.26 88.9 0)
+		(at 175.26 96.52 0)
 		(effects
 			(font
@@
 	(hierarchical_label "SWCLK"
 		(shape output)
-		(at 175.26 86.36 0)
+		(at 175.26 93.98 0)
 		(effects
 			(font
@@
 			(project "stm32-bt-board"
 				(path "/9ab97115-0b3b-4897-8d44-f79e27c270d1/0a80a0b7-1ddb-45a8-8bbe-9c16ffb72728"
-					(page "11")
+					(page "12")
 				)
 			)
@@
 			(project "stm32-bt-board"
 				(path "/9ab97115-0b3b-4897-8d44-f79e27c270d1/0a80a0b7-1ddb-45a8-8bbe-9c16ffb72728"
-					(page "12")
+					(page "10")
 				)
 			)
@@
 		)
 		(pin "SWCLK" output
-			(at 167.64 86.36 0)
+			(at 167.64 93.98 0)
 			(effects
 				(font
@@
 		)
 		(pin "SWNRST" output
-			(at 167.64 88.9 0)
+			(at 167.64 96.52 0)
 			(effects
 				(font
@@
 			(project "stm32-bt-board"
 				(path "/9ab97115-0b3b-4897-8d44-f79e27c270d1/0a80a0b7-1ddb-45a8-8bbe-9c16ffb72728"
-					(page "10")
-				)
-			)
+					(page "11")
+				)
+			)

Commit message: fix(schematic): fix connector-related errors
change uart supply from +5V to +3V3
change SWD netnames so net classes work properly
Other:
- sheet SWD ports: added SWD_NRST, SWD_SWCLK, SWD_SWDIO, SWD_SWO; removed SWCLK, SWDIO, SWNRST, SWO
Changed lines of the file:
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@@
 		)
 	)
-	(hierarchical_label "SWDIO"
+	(hierarchical_label "SWD_SWDIO"
 		(shape bidirectional)
 		(at 121.92 86.36 180)
@@
 		)
 	)
-	(hierarchical_label "SWNRST"
+	(hierarchical_label "SWD_NRST"
 		(shape output)
 		(at 175.26 96.52 0)
@@
 		)
 	)
-	(hierarchical_label "SWCLK"
+	(hierarchical_label "SWD_SWCLK"
 		(shape output)
 		(at 175.26 93.98 0)
@@
 		)
 	)
-	(hierarchical_label "SWO"
+	(hierarchical_label "SWD_SWO"
 		(shape input)
 		(at 121.92 88.9 180)
@@
 			)
 		)
-		(pin "SWCLK" output
+		(pin "SWD_SWCLK" output
 			(at 167.64 93.98 0)
 			(effects
@@
 			)
 		)
-		(pin "SWDIO" bidirectional
+		(pin "SWD_SWDIO" bidirectional
 			(at 129.54 86.36 180)
 			(effects
@@
 			)
 		)
-		(pin "SWO" input
+		(pin "SWD_SWO" input
 			(at 129.54 88.9 180)
 			(effects
@@
 			)
 		)
-		(pin "SWNRST" output
+		(pin "SWD_NRST" output
 			(at 167.64 96.52 0)
 			(effects
