File: kicad/stm32-bt-board.kicad_sch (KiCad schematic)
At the start: 0 parts

Commit message: fix(schematic): misc. fixes and stuff - sort all sheets - add the author's name to all sheets and update the date - add 0R resistor to the input of each crystal oscillator - reannotate all symbols - remove todo.md
Other:
- note added: "+3V3_LDO"
- note added: "+3V3_SWD"
- note added: "+5V_USB"
Changed lines of the file:
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@@
 	(title_block
 		(title "STM32 BT Tutorial Board")
-		(date "2026-05-27")
+		(date "2026-06-30")
 		(rev "1.0")
+		(comment 3 "Author: Odai J.")
 		(comment 4 "GitHub: https://github.com/odaij/stm32-bt-board")
 	)
@@
 		)
 	)
-	(text "+3V3"
+	(text "+3V3_LDO"
 		(exclude_from_sim no)
 		(at 88.9 91.44 0)
@@
 		)
 	)
+	(text "+3V3"
+		(exclude_from_sim no)
+		(at 165.1 86.36 0)
+		(effects
+			(font
+				(size 1.27 1.27)
+				(thickness 0.254)
+				(bold yes)
+			)
+			(justify bottom)
+		)
+	)
+	(text "+3V3"
+		(exclude_from_sim no)
+		(at 251.46 86.36 0)
+		(effects
+			(font
+				(size 1.27 1.27)
+				(thickness 0.254)
+				(bold yes)
+			)
+			(justify bottom)
+		)
+	)
 	(text "TODO:\n- assign footprints\n- finish page setup (A4, title, github repo link)\n- table of contents? block diagram? feeling fancy\n- 3V3_UART, and 3V3_SWD along with 0 ohm resistors for better netnames?"
 		(exclude_from_sim no)
@@
 		)
 	)
-	(text "+5V"
+	(text "+5V_USB"
 		(exclude_from_sim no)
 		(at 45.72 91.44 0)
@@
 		)
 	)
+	(text "+3V3_SWD"
+		(exclude_from_sim no)
+		(at 170.18 93.98 0)
+		(effects
+			(font
+				(size 1.27 1.27)
+				(thickness 0.254)
+				(bold yes)
+			)
+			(justify left)
+		)
+	)
+	(text "+5V"
+		(exclude_from_sim no)
+		(at 170.18 91.44 0)
+		(effects
+			(font
+				(size 1.27 1.27)
+				(thickness 0.254)
+				(bold yes)
+			)
+			(justify left)
+		)
+	)
 	(polyline
 		(pts
@@
 	(polyline
 		(pts
+			(xy 251.46 88.9) (xy 251.46 86.36)
+		)
+		(stroke
+			(width 0)
+			(type default)
+		)
+	)
+	(polyline
+		(pts
 			(xy -151848.5687 -151848.5687) (xy -151848.5687 -151848.5687)
 		)
@@
 	(polyline
 		(pts
+			(xy 165.1 88.9) (xy 165.1 86.36)
+		)
+		(stroke
+			(width 0)
+			(type default)
+		)
+	)
+	(polyline
+		(pts
 			(xy -151848.5687 -151848.5687) (xy -151848.5687 -151848.5687)
 		)
@@
 	(polyline
 		(pts
+			(xy 167.64 93.98) (xy 170.18 93.98)
+		)
+		(stroke
+			(width 0)
+			(type default)
+		)
+	)
+	(polyline
+		(pts
 			(xy -151848.5687 -151848.5687) (xy -151848.5687 -151848.5687)
 		)
@@
 	(polyline
 		(pts
+			(xy 170.18 91.44) (xy 167.64 91.44)
+		)
+		(stroke
+			(width 0)
+			(type default)
+		)
+	)
+	(polyline
+		(pts
 			(xy -151848.5687 -151848.5687) (xy -151848.5687 -151848.5687)
 		)
@@
 			(project "stm32-bt-board"
 				(path "/9ab97115-0b3b-4897-8d44-f79e27c270d1"
-					(page "4")
+					(page "9")
 				)
 			)
@@
 			(project "stm32-bt-board"
 				(path "/9ab97115-0b3b-4897-8d44-f79e27c270d1"
-					(page "3")
+					(page "8")
 				)
 			)

Commit message: refactor(schematic): update TODOs
Other:
- note added: "TODO: - verify footprints - finish page setup (A4, title, github repo link) - table of contents? block diagram? feeling fancy - 3V3_UART, and 3V3_SWD along with 0 ohm resistors for better netnames?"
- note removed: "TODO: - assign footprints - finish page setup (A4, title, github repo link) - table of contents? block diagram? feeling fancy - 3V3_UART, and 3V3_SWD along with 0 ohm resistors for better netnames?"
Changed lines of the file:
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@@
 		)
 	)
-	(text "TODO:\n- assign footprints\n- finish page setup (A4, title, github repo link)\n- table of contents? block diagram? feeling fancy\n- 3V3_UART, and 3V3_SWD along with 0 ohm resistors for better netnames?"
+	(text "TODO:\n- verify footprints\n- finish page setup (A4, title, github repo link)\n- table of contents? block diagram? feeling fancy\n- 3V3_UART, and 3V3_SWD along with 0 ohm resistors for better netnames?"
 		(exclude_from_sim no)
 		(at 25.4 53.34 0)

Commit message: fix(schematic): fix connector-related errors
change uart supply from +5V to +3V3
change SWD netnames so net classes work properly
Other:
- sheet Connectors ports: added SWD_NRST, SWD_SWCLK, SWD_SWDIO, SWD_SWO; removed SWCLK, SWDIO, SWNRST, SWO
Changed lines of the file:
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@@
 			)
 		)
-		(pin "SWCLK" output
+		(pin "SWD_SWCLK" output
 			(at 84.455 104.14 0)
 			(effects
@@
 			)
 		)
-		(pin "SWDIO" bidirectional
+		(pin "SWD_SWDIO" bidirectional
 			(at 46.355 104.14 180)
 			(effects
@@
 			)
 		)
-		(pin "SWO" input
+		(pin "SWD_SWO" input
 			(at 46.355 106.68 180)
 			(effects
@@
 			)
 		)
-		(pin "SWNRST" output
+		(pin "SWD_NRST" output
 			(at 84.455 106.68 0)
 			(effects
