File: kicad/stm32-bt-board.kicad_sch (KiCad schematic)
At the start: 0 parts

Commit message: feat(sch. and layout): add fiducial markers for front and back assembly
Other:
- added sheet Mechanical (mechanical.kicad_sch)
Changed lines of the file:
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@@
+	)
+	(sheet
+		(at 132.08 148.59)
+		(size 33.02 38.1)
+		(exclude_from_sim no)
+		(in_bom yes)
+		(on_board yes)
+		(dnp no)
+		(fields_autoplaced yes)
+		(stroke
+			(width 0.1524)
+			(type solid)
+		)
+		(fill
+			(color 20 20 19 1)
+		)
+		(property "Sheetname" "Mechanical"
+			(at 132.08 147.8784 0)
+			(show_name no)
+			(do_not_autoplace no)
+			(effects
+				(font
+					(size 1.27 1.27)
+				)
+				(justify left bottom)
+			)
+		)
+		(property "Sheetfile" "mechanical.kicad_sch"
+			(at 132.08 187.2746 0)
+			(show_name no)
+			(do_not_autoplace no)
+			(effects
+				(font
+					(size 1.27 1.27)
+				)
+				(justify left top)
+			)
+		)
+		(instances
+			(project "stm32-bt-board"
+				(path "/9ab97115-0b3b-4897-8d44-f79e27c270d1"
+					(page "13")
+				)
+			)
+		)
 	)
 	(sheet

Commit message: feat(BOM): fill missing parts in BOM
Other:
- note added: "TODO: - finish page setup (A4, title, github repo link) - refine root schematic - table of contents? block diagram? feeling fancy - 3V3_UART, and 3V3_SWD along with 0 ohm resistors for better netnames?"
- note removed: "TODO: - verify footprints - finish page setup (A4, title, github repo link) - table of contents? block diagram? feeling fancy - 3V3_UART, and 3V3_SWD along with 0 ohm resistors for better netnames?"
Changed lines of the file:
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@@
 		)
 	)
-	(text "TODO:\n- verify footprints\n- finish page setup (A4, title, github repo link)\n- table of contents? block diagram? feeling fancy\n- 3V3_UART, and 3V3_SWD along with 0 ohm resistors for better netnames?"
+	(text "TODO:\n- finish page setup (A4, title, github repo link)\n- refine root schematic\n- table of contents? block diagram? feeling fancy\n- 3V3_UART, and 3V3_SWD along with 0 ohm resistors for better netnames?"
 		(exclude_from_sim no)
 		(at 25.4 53.34 0)
