File: kicad/stm32-bt-board.kicad_pcb (KiCad board)
At the start: 4 copper layers, 48 x 33 mm, 60 parts, among them J1 1909763-1, J2 2171790001, J3 Conn_ARM_SWD_TagConnect_TC2030, J4 S4B-PH-K-S(LF)(SN), Q1 S9013-E, SW1 B3U-1000P, SW2 B3U-1000P, U1 MIC5365-3.3YD5, U2 USBLC6-2SC6, U3 USBLC6-2SC6, U4 STM32WB55CEU6, X1 32MHz, X2 32kHz768

Commit message: feat(manuf.): extract bom, cpl, assembly and gerbers
Parts:
- C1, C11, C18, C19, C8: value 4u7 -> (none)
- C10, C16, C17, C2, C20, C21, C3, C4, C5, C6, C7, C9: value 100n -> (none)
- C12: value 0p8 -> (none)
- C13: value 0p3 -> (none)
- C14, C15: value 10p -> (none)
- D1: value VLMB1500-GS08 -> (none)
- D2: value BAT54K -> (none)
- D3: value VLMS1500-GS08 -> (none)
- FID1, FID2, FID3: value Fiducial -> (none)
- FL1: value DLF162500LT-5028A1 -> (none)
- J1: value 1909763-1 -> (none)
- J2: value 2171790001 -> (none)
- J3: value Conn_ARM_SWD_TagConnect_TC2030 -> (none)
- J4: value S4B-PH-K-S(LF)(SN) -> (none)
- L1: value 10n -> (none)
- L2: value 10u -> (none)
- L3: value 2n7 -> (none)
- Q1: value S9013-E -> (none)
- R1, R2, R3: value 0R -> (none)
- R10, R11, R4, R7: value 220R -> (none)
- R13, R16, R5, R8, R9: value 5k1 -> (none)
- R6: value 100k -> (none)
- SW1, SW2: value B3U-1000P -> (none)
- U1: value MIC5365-3.3YD5 -> (none)
- U2, U3: value USBLC6-2SC6 -> (none)
- U4: value STM32WB55CEU6 -> (none)
- X1: value 32MHz -> (none)
- X2: value 32kHz768 -> (none)
Other:
- rule pad_to_mask_clearance: 0.01 -> 0
