File: kicad/connectors_swd.kicad_sch (KiCad schematic)
At the start: 2 parts, among them J2 Conn_ARM_SWD_TagConnect_TC2030

Commit message: fix(schematic): misc. fixes and stuff - sort all sheets - add the author's name to all sheets and update the date - add 0R resistor to the input of each crystal oscillator - reannotate all symbols - remove todo.md
Parts:
- renumbered C21 to C20, J2 to J3
Changed lines of the file:
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@@
 	(generator_version "10.0")
 	(paper "A4")
+	(title_block
+		(date "2026-06-30")
+		(rev "1.0")
+		(comment 3 "Author: Odai J.")
+		(comment 4 "GitHub: https://github.com/odaij/stm32-bt-board")
+	)
 	(rectangle
 		(start 114.3 76.2)
@@
 		(dnp no)
 		(fields_autoplaced yes)
-		(property "Reference" "#PWR012"
+		(property "Reference" "#PWR033"
 			(at 161.29 96.52 0)
 			(hide yes)
@@
 			(project "stm32-bt-board"
 				(path "/9ab97115-0b3b-4897-8d44-f79e27c270d1/0a80a0b7-1ddb-45a8-8bbe-9c16ffb72728/e6e5b388-18a0-444d-846c-ffc05907a441"
-					(reference "#PWR012")
+					(reference "#PWR033")
 					(unit 1)
 				)
@@
 		(dnp no)
 		(fields_autoplaced yes)
-		(property "Reference" "C21"
+		(property "Reference" "C20"
 			(at 163.83 86.3662 0)
 			(show_name no)
@@
 			(project "stm32-bt-board"
 				(path "/9ab97115-0b3b-4897-8d44-f79e27c270d1/0a80a0b7-1ddb-45a8-8bbe-9c16ffb72728/e6e5b388-18a0-444d-846c-ffc05907a441"
-					(reference "C21")
+					(reference "C20")
 					(unit 1)
 				)
@@
 		(dnp no)
 		(fields_autoplaced yes)
-		(property "Reference" "#PWR06"
+		(property "Reference" "#PWR034"
 			(at 154.94 119.38 0)
 			(hide yes)
@@
 			(project "stm32-bt-board"
 				(path "/9ab97115-0b3b-4897-8d44-f79e27c270d1/0a80a0b7-1ddb-45a8-8bbe-9c16ffb72728/e6e5b388-18a0-444d-846c-ffc05907a441"
-					(reference "#PWR06")
+					(reference "#PWR034")
 					(unit 1)
 				)
@@
 		(dnp no)
 		(fields_autoplaced yes)
-		(property "Reference" "J2"
+		(property "Reference" "J3"
 			(at 151.13 100.3299 0)
 			(show_name no)
@@
 			(project "stm32-bt-board"
 				(path "/9ab97115-0b3b-4897-8d44-f79e27c270d1/0a80a0b7-1ddb-45a8-8bbe-9c16ffb72728/e6e5b388-18a0-444d-846c-ffc05907a441"
-					(reference "J2")
+					(reference "J3")
 					(unit 1)
 				)
@@
 		(dnp no)
 		(fields_autoplaced yes)
-		(property "Reference" "#PWR09"
+		(property "Reference" "#PWR032"
 			(at 154.94 87.63 0)
 			(hide yes)
@@
 			(project "stm32-bt-board"
 				(path "/9ab97115-0b3b-4897-8d44-f79e27c270d1/0a80a0b7-1ddb-45a8-8bbe-9c16ffb72728/e6e5b388-18a0-444d-846c-ffc05907a441"
-					(reference "#PWR09")
+					(reference "#PWR032")
 					(unit 1)
 				)

Commit message: everything: select real components, refactor schematic, add a user-led driving circuit, and more
Parts:
- C20: footprint (none) -> Capacitor_SMD:C_0402_1005Metric; Distributor (none) -> LCSC; Distributor Link (none) -> https://www.lcsc.com/product-detail/C60474.html?s_z=s_p_CC0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; MPN (none) -> CC0402KRX7R7BB104; Manufacturer (none) -> YAGEO
Changed lines of the file:
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@@
 			)
 		)
-		(property "Footprint" ""
-			(at 161.29 87.63 0)
-			(hide yes)
-			(show_name no)
-			(do_not_autoplace no)
-			(effects
-				(font
-					(size 1.27 1.27)
-				)
-			)
-		)
-		(property "Datasheet" ""
-			(at 161.29 87.63 0)
-			(hide yes)
-			(show_name no)
-			(do_not_autoplace no)
-			(effects
-				(font
-					(size 1.27 1.27)
-				)
-			)
-		)
-		(property "Description" "Unpolarized capacitor, small symbol"
+		(property "Footprint" "Capacitor_SMD:C_0402_1005Metric"
+			(at 161.29 87.63 0)
+			(hide yes)
+			(show_name no)
+			(do_not_autoplace no)
+			(effects
+				(font
+					(size 1.27 1.27)
+				)
+			)
+		)
+		(property "Datasheet" "https://www.lcsc.com/datasheet/C60474.pdf?spm=wm.sxq.inf.ggs___wm.fly.bg.0.xh&lcsc_vid=RlRYUFFURFcNVFIDFVMMXgZSRlJeUABSQVNfAwJfQwIxVlNeTldcUFdQQFNXVTsOAxUeFF5JWBYZEEoKFBINSQcJGk4NBhADEA4cHktXRlVcSQwSGg0%3D"
+			(at 161.29 87.63 0)
+			(hide yes)
+			(show_name no)
+			(do_not_autoplace no)
+			(effects
+				(font
+					(size 1.27 1.27)
+				)
+			)
+		)
+		(property "Description" "CAP CER 100nF 16V X7R 0402"
 			(at 161.29 87.63 0)
 			(hide yes)
@@
 			)
 		)
-		(property "Distributor Link" ""
-			(at 161.29 87.63 0)
-			(hide yes)
-			(show_name no)
-			(do_not_autoplace no)
-			(effects
-				(font
-					(size 1.27 1.27)
-				)
-			)
-		)
-		(property "Manufacturer" ""
-			(at 161.29 87.63 0)
-			(hide yes)
-			(show_name no)
-			(do_not_autoplace no)
-			(effects
-				(font
-					(size 1.27 1.27)
-				)
-			)
-		)
-		(property "Manufacturer Part Number" ""
+		(property "Distributor Link" "https://www.lcsc.com/product-detail/C60474.html?s_z=s_p_CC0402KRX7R7BB104&spm=wm.fly.bg.0.xh&lcsc_vid=RlRYUFFURFcNVFIDFVMMXgZSRlJeUABSQVNfAwJfQwIxVlNeTldcUFdQQFNXVTsOAxUeFF5JWBYZEEoKFBINSQcJGk4NBhADEA4cHktXRlVcSQwSGg0%3D"
+			(at 161.29 87.63 0)
+			(hide yes)
+			(show_name no)
+			(do_not_autoplace no)
+			(effects
+				(font
+					(size 1.27 1.27)
+				)
+			)
+		)
+		(property "Manufacturer" "YAGEO"
+			(at 161.29 87.63 0)
+			(hide yes)
+			(show_name no)
+			(do_not_autoplace no)
+			(effects
+				(font
+					(size 1.27 1.27)
+				)
+			)
+		)
+		(property "Distributor" "LCSC"
+			(at 161.29 87.63 0)
+			(hide yes)
+			(show_name no)
+			(do_not_autoplace no)
+			(effects
+				(font
+					(size 1.27 1.27)
+				)
+			)
+		)
+		(property "MPN" "CC0402KRX7R7BB104"
 			(at 161.29 87.63 0)
 			(hide yes)
@@
 			)
 		)
-		(property "Manufacturer Part Number" ""
-			(at 157.48 101.6 0)
-			(hide yes)
+		(property "Distributor" ""
+			(at 157.48 101.6 0)
+			(hide yes)

Commit message: fix(footprints and symbols): add missing footprints and symbols
Parts:
- J3: Distributor (none) -> LCSC
Changed lines of the file:
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@@
 			)
 		)
-		(property "Distributor" ""
+		(property "Distributor" "LCSC"
 			(at 157.48 101.6 0)
 			(hide yes)

Commit message: fix(schematic): fix connector-related errors
change uart supply from +5V to +3V3
change SWD netnames so net classes work properly
Connections:
- net SWCLK renamed SWD_SWCLK
- net SWDIO renamed SWD_SWDIO
- net SWNRST renamed SWD_NRST
- net SWO renamed SWD_SWO
Changed lines of the file:
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@@
 		)
 	)
-	(hierarchical_label "SWCLK"
+	(hierarchical_label "SWD_SWCLK"
 		(shape output)
 		(at 172.72 101.6 0)
@@
 		)
 	)
-	(hierarchical_label "SWNRST"
+	(hierarchical_label "SWD_NRST"
 		(shape output)
 		(at 172.72 96.52 0)
@@
 		)
 	)
-	(hierarchical_label "SWO"
+	(hierarchical_label "SWD_SWO"
 		(shape input)
 		(at 172.72 106.68 0)
@@
 		)
 	)
-	(hierarchical_label "SWDIO"
+	(hierarchical_label "SWD_SWDIO"
 		(shape bidirectional)
 		(at 172.72 104.14 0)

Commit message: feat(BOM): fill missing parts in BOM
Parts:
- J3: Distributor LCSC -> (none)
Changed lines of the file:
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@@
 			)
 		)
-		(property "Distributor" "LCSC"
+		(property "Distributor" ""
 			(at 157.48 101.6 0)
 			(hide yes)

Commit message: feat(manuf.): edit BOM and CPL to match JLCPCB's requirements
however, please pay close attention to the rotations during ordering, especially for the SOT components, as JLCPCB messes them up a bit, same for the connector and the filter
Parts:
- C20: Distributor Link https://www.lcsc.com/product-detail/C60474.html?s_z=s_p_CC0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 -> https://www.lcsc.com/product-detail/C60474.html; JLCPCB Part # (none) -> C60474
Changed lines of the file:
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@@
-			)
-		)
-		(property "Distributor Link" "https://www.lcsc.com/product-detail/C60474.html?s_z=s_p_CC0402KRX7R7BB104&spm=wm.fly.bg.0.xh&lcsc_vid=RlRYUFFURFcNVFIDFVMMXgZSRlJeUABSQVNfAwJfQwIxVlNeTldcUFdQQFNXVTsOAxUeFF5JWBYZEEoKFBINSQcJGk4NBhADEA4cHktXRlVcSQwSGg0%3D"
-			(at 161.29 87.63 0)
-			(hide yes)
-			(show_name no)
-			(do_not_autoplace no)
-			(effects
-				(font
-					(size 1.27 1.27)
-				)
 			)
 		)
@@
 		)
 		(property "MPN" "CC0402KRX7R7BB104"
+			(at 161.29 87.63 0)
+			(hide yes)
+			(show_name no)
+			(do_not_autoplace no)
+			(effects
+				(font
+					(size 1.27 1.27)
+				)
+			)
+		)
+		(property "JLCPCB Part #" "C60474"
+			(at 161.29 87.63 0)
+			(hide yes)
+			(show_name no)
+			(do_not_autoplace no)
+			(effects
+				(font
+					(size 1.27 1.27)
+				)
+			)
+		)
+		(property "Distributor Link" "https://www.lcsc.com/product-detail/C60474.html"
 			(at 161.29 87.63 0)
 			(hide yes)
@@
 			)
 		)
-		(property "Distributor Link" ""
-			(at 157.48 101.6 0)
-			(hide yes)
-			(show_name no)
-			(do_not_autoplace no)
-			(effects
-				(font
-					(size 1.27 1.27)
-				)
-			)
-		)
 		(property "Manufacturer" ""
 			(at 157.48 101.6 0)
@@
 			(at 157.48 101.6 0)
 			(hide yes)
+			(show_name no)
+			(do_not_autoplace no)
+			(effects
+				(font
+					(size 1.27 1.27)
+				)
+			)
+		)
+		(property "JLCPCB Part #" ""
+			(at 157.48 101.6 0)
+			(hide yes)
