File: kicad/connectors_uart.kicad_sch (KiCad schematic)
At the start: 5 parts, among them J4 Conn_01x04_Pin, U4 USBLC6-2SC6

Commit message: fix(schematic): misc. fixes and stuff - sort all sheets - add the author's name to all sheets and update the date - add 0R resistor to the input of each crystal oscillator - reannotate all symbols - remove todo.md
Parts:
- renumbered C20 to C21, R6 to R10, R5 to R11, U4 to U3
Changed lines of the file:
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@@
 	(generator_version "10.0")
 	(paper "A4")
+	(title_block
+		(date "2026-06-30")
+		(rev "1.0")
+		(comment 3 "Author: Odai J.")
+		(comment 4 "GitHub: https://github.com/odaij/stm32-bt-board")
+	)
 	(rectangle
 		(start 101.6 76.2)
@@
 		(in_pos_files yes)
 		(dnp no)
-		(property "Reference" "U4"
+		(property "Reference" "U3"
 			(at 148.336 90.17 0)
 			(show_name no)
@@
 			(project "stm32-bt-board"
 				(path "/9ab97115-0b3b-4897-8d44-f79e27c270d1/0a80a0b7-1ddb-45a8-8bbe-9c16ffb72728/361c8e35-3db7-4e84-96f3-a18e08b55d73"
-					(reference "U4")
+					(reference "U3")
 					(unit 1)
 				)
@@
 		(dnp no)
 		(fields_autoplaced yes)
-		(property "Reference" "#PWR033"
+		(property "Reference" "#PWR035"
 			(at 123.19 87.63 0)
 			(hide yes)
@@
 			(project "stm32-bt-board"
 				(path "/9ab97115-0b3b-4897-8d44-f79e27c270d1/0a80a0b7-1ddb-45a8-8bbe-9c16ffb72728/361c8e35-3db7-4e84-96f3-a18e08b55d73"
-					(reference "#PWR033")
+					(reference "#PWR035")
 					(unit 1)
 				)
@@
 		(in_pos_files yes)
 		(dnp no)
-		(property "Reference" "R6"
+		(property "Reference" "R10"
 			(at 179.324 98.806 90)
 			(show_name no)
@@
 			(project "stm32-bt-board"
 				(path "/9ab97115-0b3b-4897-8d44-f79e27c270d1/0a80a0b7-1ddb-45a8-8bbe-9c16ffb72728/361c8e35-3db7-4e84-96f3-a18e08b55d73"
-					(reference "R6")
+					(reference "R10")
 					(unit 1)
 				)
@@
 		(dnp no)
 		(fields_autoplaced yes)
-		(property "Reference" "C20"
+		(property "Reference" "C21"
 			(at 129.54 88.9062 0)
 			(show_name no)
@@
 			(project "stm32-bt-board"
 				(path "/9ab97115-0b3b-4897-8d44-f79e27c270d1/0a80a0b7-1ddb-45a8-8bbe-9c16ffb72728/361c8e35-3db7-4e84-96f3-a18e08b55d73"
-					(reference "C20")
+					(reference "C21")
 					(unit 1)
 				)
@@
 		(in_pos_files yes)
 		(dnp no)
-		(property "Reference" "R5"
+		(property "Reference" "R11"
 			(at 179.324 106.934 90)
 			(show_name no)
@@
 			(project "stm32-bt-board"
 				(path "/9ab97115-0b3b-4897-8d44-f79e27c270d1/0a80a0b7-1ddb-45a8-8bbe-9c16ffb72728/361c8e35-3db7-4e84-96f3-a18e08b55d73"
-					(reference "R5")
+					(reference "R11")
 					(unit 1)
 				)
@@
 		(dnp no)
 		(fields_autoplaced yes)
-		(property "Reference" "#PWR034"
+		(property "Reference" "#PWR038"
 			(at 123.19 116.84 0)
 			(hide yes)
@@
 			(project "stm32-bt-board"
 				(path "/9ab97115-0b3b-4897-8d44-f79e27c270d1/0a80a0b7-1ddb-45a8-8bbe-9c16ffb72728/361c8e35-3db7-4e84-96f3-a18e08b55d73"
-					(reference "#PWR034")
+					(reference "#PWR038")
 					(unit 1)
 				)
@@
 		(dnp no)
 		(fields_autoplaced yes)
-		(property "Reference" "#PWR035"
+		(property "Reference" "#PWR036"
 			(at 146.05 99.06 0)
 			(hide yes)
@@
 			(project "stm32-bt-board"
 				(path "/9ab97115-0b3b-4897-8d44-f79e27c270d1/0a80a0b7-1ddb-45a8-8bbe-9c16ffb72728/361c8e35-3db7-4e84-96f3-a18e08b55d73"
-					(reference "#PWR035")
+					(reference "#PWR036")
 					(unit 1)
 				)
@@
 		(dnp no)
 		(fields_autoplaced yes)
-		(property "Reference" "#PWR036"
+		(property "Reference" "#PWR039"
 			(at 146.05 116.84 0)
 			(hide yes)
@@
 			(project "stm32-bt-board"
 				(path "/9ab97115-0b3b-4897-8d44-f79e27c270d1/0a80a0b7-1ddb-45a8-8bbe-9c16ffb72728/361c8e35-3db7-4e84-96f3-a18e08b55d73"
-					(reference "#PWR036")
+					(reference "#PWR039")
 					(unit 1)
 				)

Commit message: everything: select real components, refactor schematic, add a user-led driving circuit, and more
Parts:
- C21: footprint (none) -> Capacitor_SMD:C_0402_1005Metric; Distributor (none) -> LCSC; Distributor Link (none) -> https://www.lcsc.com/product-detail/C60474.html?s_z=s_p_CC0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; MPN (none) -> CC0402KRX7R7BB104; Manufacturer (none) -> YAGEO
- J4: footprint (none) -> Connector_PinHeader_2.54mm:PinHeader_1x04_P2.54mm_Vertical
- R10, R11: footprint (none) -> Resistor_SMD:R_0402_1005Metric
- U3: Distributor (none) -> LCSC; Distributor Link (none) -> https://www.lcsc.com/product-detail/C7519.html?s_z=s_p_USBL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; MPN (none) -> USBLC6-2SC6; Manufacturer (none) -> ST
Changed lines of the file:
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@@
 			)
 		)
-		(property "Distributor Link" ""
+		(property "Distributor Link" "https://www.lcsc.com/product-detail/C7519.html?s_z=s_p_USBLC6-2SC6&spm=wm.fly.bg.0.xh&lcsc_vid=RlRYUFFURFcNVFIDFVMMXgZSRlJeUABSQVNfAwJfQwIxVlNeTlddV1JTQlFfUDsOAxUeFF5JWBYZEEoKFBINSQcJGk4eFQsCAgIaSgADAwAHC0slQVNYV11eWQkaCgg%3D"
 			(at 146.05 101.6 0)
 			(hide yes)
@@
 			)
 		)
-		(property "Manufacturer" ""
+		(property "Manufacturer" "ST"
 			(at 146.05 101.6 0)
 			(hide yes)
@@
 			)
 		)
-		(property "Manufacturer Part Number" ""
+		(property "Distributor" "LCSC"
+			(at 146.05 101.6 0)
+			(hide yes)
+			(show_name no)
+			(do_not_autoplace no)
+			(effects
+				(font
+					(size 1.27 1.27)
+				)
+			)
+		)
+		(property "MPN" "USBLC6-2SC6"
 			(at 146.05 101.6 0)
 			(hide yes)
@@
 			)
 		)
-		(property "Footprint" ""
+		(property "Footprint" "Resistor_SMD:R_0402_1005Metric"
 			(at 179.07 99.822 90)
 			(hide yes)
@@
 			)
 		)
-		(property "Manufacturer Part Number" ""
+		(property "Distributor" ""
 			(at 179.07 101.6 90)
 			(hide yes)
@@
 			)
 		)
-		(property "Footprint" ""
-			(at 127 90.17 0)
-			(hide yes)
-			(show_name no)
-			(do_not_autoplace no)
-			(effects
-				(font
-					(size 1.27 1.27)
-				)
-			)
-		)
-		(property "Datasheet" ""
-			(at 127 90.17 0)
-			(hide yes)
-			(show_name no)
-			(do_not_autoplace no)
-			(effects
-				(font
-					(size 1.27 1.27)
-				)
-			)
-		)
-		(property "Description" "Unpolarized capacitor, small symbol"
+		(property "Footprint" "Capacitor_SMD:C_0402_1005Metric"
+			(at 127 90.17 0)
+			(hide yes)
+			(show_name no)
+			(do_not_autoplace no)
+			(effects
+				(font
+					(size 1.27 1.27)
+				)
+			)
+		)
+		(property "Datasheet" "https://www.lcsc.com/datasheet/C60474.pdf?spm=wm.sxq.inf.ggs___wm.fly.bg.0.xh&lcsc_vid=RlRYUFFURFcNVFIDFVMMXgZSRlJeUABSQVNfAwJfQwIxVlNeTldcUFdQQFNXVTsOAxUeFF5JWBYZEEoKFBINSQcJGk4NBhADEA4cHktXRlVcSQwSGg0%3D"
+			(at 127 90.17 0)
+			(hide yes)
+			(show_name no)
+			(do_not_autoplace no)
+			(effects
+				(font
+					(size 1.27 1.27)
+				)
+			)
+		)
+		(property "Description" "CAP CER 100nF 16V X7R 0402"
 			(at 127 90.17 0)
 			(hide yes)
@@
 			)
 		)
-		(property "Distributor Link" ""
-			(at 127 90.17 0)
-			(hide yes)
-			(show_name no)
-			(do_not_autoplace no)
-			(effects
-				(font
-					(size 1.27 1.27)
-				)
-			)
-		)
-		(property "Manufacturer" ""
-			(at 127 90.17 0)
-			(hide yes)
-			(show_name no)
-			(do_not_autoplace no)
-			(effects
-				(font
-					(size 1.27 1.27)
-				)
-			)
-		)
-		(property "Manufacturer Part Number" ""
+		(property "Distributor Link" "https://www.lcsc.com/product-detail/C60474.html?s_z=s_p_CC0402KRX7R7BB104&spm=wm.fly.bg.0.xh&lcsc_vid=RlRYUFFURFcNVFIDFVMMXgZSRlJeUABSQVNfAwJfQwIxVlNeTldcUFdQQFNXVTsOAxUeFF5JWBYZEEoKFBINSQcJGk4NBhADEA4cHktXRlVcSQwSGg0%3D"
+			(at 127 90.17 0)
+			(hide yes)
+			(show_name no)
+			(do_not_autoplace no)
+			(effects
+				(font
+					(size 1.27 1.27)
+				)
+			)
+		)
+		(property "Manufacturer" "YAGEO"
+			(at 127 90.17 0)
+			(hide yes)
+			(show_name no)
+			(do_not_autoplace no)
+			(effects
+				(font
+					(size 1.27 1.27)
+				)
+			)
+		)
+		(property "Distributor" "LCSC"
+			(at 127 90.17 0)
+			(hide yes)
+			(show_name no)
+			(do_not_autoplace no)
+			(effects
+				(font
+					(size 1.27 1.27)
+				)
+			)
+		)
+		(property "MPN" "CC0402KRX7R7BB104"
 			(at 127 90.17 0)
 			(hide yes)
@@
 			)
 		)
-		(property "Footprint" ""
+		(property "Footprint" "Connector_PinHeader_2.54mm:PinHeader_1x04_P2.54mm_Vertical"
 			(at 109.22 101.6 0)
 			(hide yes)
@@
 			)
 		)
-		(property "Manufacturer Part Number" ""
+		(property "Distributor" ""
 			(at 109.22 101.6 0)
 			(hide yes)
@@
 			)
 		)
-		(property "Footprint" ""
+		(property "Footprint" "Resistor_SMD:R_0402_1005Metric"
 			(at 179.07 105.918 90)
 			(hide yes)
@@
 			)
 		)
-		(property "Manufacturer Part Number" ""
+		(property "Distributor" ""
 			(at 179.07 104.14 90)
 			(hide yes)

Commit message: fix(footprints and symbols): add missing footprints and symbols
Parts:
- removed J4: Conn_01x04_Pin, Connector_PinHeader_2.54mm:PinHeader_1x04_P2.54mm_Vertical, symbol Connector:Conn_01x04_Pin
- added J4: S4B-PH-K-S(LF)(SN), #stm32-bt-board-external-footprints:S4B-PH-K-S(LF)(SN), symbol #stm32-bt-board-external-symbols:S4B-PH-K-S(LF)(SN)
Connections:
- net +3V3: now also J4.1 (Pin_1)
- net GND: now also J4.4 (Pin_4)
- net UART_CON_RX: now also J4.2 (Pin_2)
- net UART_CON_TX: now also J4.3 (Pin_3)
Changed lines of the file:
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@@
 	)
 	(rectangle
-		(start 101.6 76.2)
+		(start 97.79 76.2)
 		(end 199.39 115.57)
 		(stroke
@@
 	)
 	(symbol
-		(lib_id "Connector:Conn_01x04_Pin")
+		(lib_id "#stm32-bt-board-external-symbols:S4B-PH-K-S(LF)(SN)")
 		(at 109.22 101.6 0)
 		(unit 1)
@@
 			)
 		)
-		(property "Value" "Conn_01x04_Pin"
+		(property "Value" "S4B-PH-K-S(LF)(SN)"
 			(at 109.855 96.52 0)
 			(show_name no)
@@
 			)
 		)
-		(property "Footprint" "Connector_PinHeader_2.54mm:PinHeader_1x04_P2.54mm_Vertical"
+		(property "Footprint" "#stm32-bt-board-external-footprints:S4B-PH-K-S(LF)(SN)"
 			(at 109.22 101.6 0)
 			(hide yes)
@@
 			)
 		)
-		(property "Datasheet" ""
+		(property "Datasheet" "https://www.lcsc.com/datasheet/C157926.pdf?spm=wm.sxq.inf.ggs___wm.fly.bg.0.xh&lcsc_vid=RlRYUFFURFcNVFIDFVMMXgZSRlJeUABSQVNfAwJfQwIxVlNeTllXUl1SRlVdUjsOAxUeFF5JWBYZEEoKFBINSQcJGk4eFQsCAgIaSgADAwAHC0slRVJfVFZfWQkaCgg%3D"
 			(at 109.22 101.6 0)
 			(hide yes)
@@
 			)
 		)
-		(property "Description" "Generic connector, single row, 01x04, script generated"
+		(property "Description" "CONN HEADER TH R/A 4POS 2mm"
 			(at 109.22 101.6 0)
 			(hide yes)
@@
 			)
 		)
-		(property "KLC_S3.3" ""
+		(property "Distributor" "LCSC"
 			(at 109.22 101.6 0)
 			(hide yes)
@@
 			)
 		)
-		(property "KLC_S4.1" ""
-			(at 109.22 101.6 0)
-			(hide yes)
-			(show_name no)
-			(do_not_autoplace no)
-			(effects
-				(font
-					(size 1.27 1.27)
-				)
-			)
-		)
-		(property "Distributor Link" ""
-			(at 109.22 101.6 0)
-			(hide yes)
-			(show_name no)
-			(do_not_autoplace no)
-			(effects
-				(font
-					(size 1.27 1.27)
-				)
-			)
-		)
-		(property "Manufacturer" ""
-			(at 109.22 101.6 0)
-			(hide yes)
-			(show_name no)
-			(do_not_autoplace no)
-			(effects
-				(font
-					(size 1.27 1.27)
-				)
-			)
-		)
-		(property "Distributor" ""
-			(at 109.22 101.6 0)
-			(hide yes)
-			(show_name no)
-			(do_not_autoplace no)
-			(effects
-				(font
-					(size 1.27 1.27)
-				)
-			)
+		(pin "3"
+		)
+		(pin "4"
 		)
 		(pin "1"
@@
 		(pin "2"
 		)
-		(pin "3"
-		)
-		(pin "4"
-		)
 		(instances

Commit message: fix(schematic): fix connector-related errors
change uart supply from +5V to +3V3
change SWD netnames so net classes work properly
Connections:
- net +5V is gone; now on net +3V3: U3.5 (VBUS)
Changed lines of the file:
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@@
 		(in_pos_files yes)
 		(dnp no)
-		(fields_autoplaced yes)
 		(property "Reference" "#PWR036"
 			(at 146.05 99.06 0)
@@
 			)
 		)
-		(property "Value" "+5V"
-			(at 146.05 90.17 0)
+		(property "Value" "+3V3"
+			(at 142.24 91.44 0)
 			(show_name no)
 			(do_not_autoplace no)
@@
 					(size 1.27 1.27)
 				)
+				(justify left)
 			)
 		)

Commit message: feat(BOM): fill missing parts in BOM
Parts:
- J4: Distributor Link (none) -> https://www.lcsc.com/product-detail/C157926.html?s_z=s_p_S4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; MPN (none) -> S4B-PH-K-S(LF)(SN); Manufacturer (none) -> JST
- R10, R11: Distributor (none) -> LCSC; Distributor Link (none) -> https://www.lcsc.com/product-detail/C2909336.html; MPN (none) -> FRC0402F2200TS; Manufacturer (none) -> FOJAN
Changed lines of the file:
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@@
 			)
 		)
-		(property "Datasheet" ""
+		(property "Datasheet" "https://www.lcsc.com/datasheet/C2909336.pdf"
 			(at 179.07 101.6 0)
 			(hide yes)
@@
 			)
 		)
-		(property "Description" "Resistor"
+		(property "Description" "RES 220Ω ±1% 62.5mW 0402"
 			(at 179.07 101.6 0)
 			(hide yes)
@@
 			)
 		)
-		(property "Distributor Link" ""
-			(at 179.07 101.6 90)
-			(hide yes)
-			(show_name no)
-			(do_not_autoplace no)
-			(effects
-				(font
-					(size 1.27 1.27)
-				)
-			)
-		)
-		(property "Manufacturer" ""
-			(at 179.07 101.6 90)
-			(hide yes)
-			(show_name no)
-			(do_not_autoplace no)
-			(effects
-				(font
-					(size 1.27 1.27)
-				)
-			)
-		)
-		(property "Distributor" ""
+		(property "Distributor Link" "https://www.lcsc.com/product-detail/C2909336.html"
+			(at 179.07 101.6 90)
+			(hide yes)
+			(show_name no)
+			(do_not_autoplace no)
+			(effects
+				(font
+					(size 1.27 1.27)
+				)
+			)
+		)
+		(property "Manufacturer" "FOJAN"
+			(at 179.07 101.6 90)
+			(hide yes)
+			(show_name no)
+			(do_not_autoplace no)
+			(effects
+				(font
+					(size 1.27 1.27)
+				)
+			)
+		)
+		(property "Distributor" "LCSC"
+			(at 179.07 101.6 90)
+			(hide yes)
+			(show_name no)
+			(do_not_autoplace no)
+			(effects
+				(font
+					(size 1.27 1.27)
+				)
+			)
+		)
+		(property "MPN" "FRC0402F2200TS"
 			(at 179.07 101.6 90)
 			(hide yes)
@@
 			)
 		)
+		(property "Distributor Link" "https://www.lcsc.com/product-detail/C157926.html?s_z=s_p_S4B-PH-K-S%28LF%29%28SN%29"
+			(at 109.22 101.6 0)
+			(hide yes)
+			(show_name no)
+			(do_not_autoplace no)
+			(effects
+				(font
+					(size 1.27 1.27)
+				)
+			)
+		)
+		(property "MPN" "S4B-PH-K-S(LF)(SN)"
+			(at 109.22 101.6 0)
+			(hide yes)
+			(show_name no)
+			(do_not_autoplace no)
+			(effects
+				(font
+					(size 1.27 1.27)
+				)
+			)
+		)
+		(property "Manufacturer" "JST"
+			(at 109.22 101.6 0)
+			(hide yes)
+			(show_name no)
+			(do_not_autoplace no)
+			(effects
+				(font
+					(size 1.27 1.27)
+				)
+			)
+		)
 		(pin "3"
 		)
@@
 			)
 		)
-		(property "Datasheet" ""
+		(property "Datasheet" "https://www.lcsc.com/datasheet/C2909336.pdf"
 			(at 179.07 104.14 0)
 			(hide yes)
@@
 			)
 		)
-		(property "Description" "Resistor"
+		(property "Description" "RES 220Ω ±1% 62.5mW 0402"
 			(at 179.07 104.14 0)
 			(hide yes)
@@
 			)
 		)
-		(property "Distributor Link" ""
-			(at 179.07 104.14 90)
-			(hide yes)
-			(show_name no)
-			(do_not_autoplace no)
-			(effects
-				(font
-					(size 1.27 1.27)
-				)
-			)
-		)
-		(property "Manufacturer" ""
-			(at 179.07 104.14 90)
-			(hide yes)
-			(show_name no)
-			(do_not_autoplace no)
-			(effects
-				(font
-					(size 1.27 1.27)
-				)
-			)
-		)
-		(property "Distributor" ""
-			(at 179.07 104.14 90)
-			(hide yes)
+		(property "Distributor Link" "https://www.lcsc.com/product-detail/C2909336.html"
+			(at 179.07 104.14 90)
+			(hide yes)
+			(show_name no)
+			(do_not_autoplace no)
+			(effects
+				(font
+					(size 1.27 1.27)
+				)
+			)
+		)
+		(property "Manufacturer" "FOJAN"
+			(at 179.07 104.14 90)
+			(hide yes)
+			(show_name no)
+			(do_not_autoplace no)
+			(effects
+				(font
+					(size 1.27 1.27)
+				)
+			)
+		)
+		(property "Distributor" "LCSC"
+			(at 179.07 104.14 90)
+			(hide yes)
+			(show_name no)
+			(do_not_autoplace no)
+			(effects
+				(font
+					(size 1.27 1.27)
+				)
+			)
+		)
+		(property "MPN" "FRC0402F2200TS"
+			(at 179.07 104.14 90)
+			(hide yes)

Commit message: feat(manuf.): edit BOM and CPL to match JLCPCB's requirements
however, please pay close attention to the rotations during ordering, especially for the SOT components, as JLCPCB messes them up a bit, same for the connector and the filter
Parts:
- C21: Distributor Link https://www.lcsc.com/product-detail/C60474.html?s_z=s_p_CC0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 -> https://www.lcsc.com/product-detail/C60474.html; JLCPCB Part # (none) -> C60474
- J4: Distributor Link https://www.lcsc.com/product-detail/C157926.html?s_z=s_p_S4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 -> https://www.lcsc.com/product-detail/C157926.html; JLCPCB Part # (none) -> C157926
- R10, R11: JLCPCB Part # (none) -> C2909336
- U3: Distributor Link https://www.lcsc.com/product-detail/C7519.html?s_z=s_p_USBL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 -> https://www.lcsc.com/product-detail/C7519.html; JLCPCB Part # (none) -> C7519
Changed lines of the file:
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@@
-			)
-		)
-		(property "Distributor Link" "https://www.lcsc.com/product-detail/C7519.html?s_z=s_p_USBLC6-2SC6&spm=wm.fly.bg.0.xh&lcsc_vid=RlRYUFFURFcNVFIDFVMMXgZSRlJeUABSQVNfAwJfQwIxVlNeTlddV1JTQlFfUDsOAxUeFF5JWBYZEEoKFBINSQcJGk4eFQsCAgIaSgADAwAHC0slQVNYV11eWQkaCgg%3D"
-			(at 146.05 101.6 0)
-			(hide yes)
-			(show_name no)
-			(do_not_autoplace no)
-			(effects
-				(font
-					(size 1.27 1.27)
-				)
 			)
 		)
@@
 		)
 		(property "MPN" "USBLC6-2SC6"
+			(at 146.05 101.6 0)
+			(hide yes)
+			(show_name no)
+			(do_not_autoplace no)
+			(effects
+				(font
+					(size 1.27 1.27)
+				)
+			)
+		)
+		(property "JLCPCB Part #" "C7519"
+			(at 146.05 101.6 0)
+			(hide yes)
+			(show_name no)
+			(do_not_autoplace no)
+			(effects
+				(font
+					(size 1.27 1.27)
+				)
+			)
+		)
+		(property "Distributor Link" "https://www.lcsc.com/product-detail/C7519.html"
 			(at 146.05 101.6 0)
 			(hide yes)
@@
 			)
 		)
-		(property "Distributor Link" "https://www.lcsc.com/product-detail/C2909336.html"
-			(at 179.07 101.6 90)
-			(hide yes)
-			(show_name no)
-			(do_not_autoplace no)
-			(effects
-				(font
-					(size 1.27 1.27)
-				)
-			)
-		)
 		(property "Manufacturer" "FOJAN"
 			(at 179.07 101.6 90)
@@
 		)
 		(property "MPN" "FRC0402F2200TS"
+			(at 179.07 101.6 90)
+			(hide yes)
+			(show_name no)
+			(do_not_autoplace no)
+			(effects
+				(font
+					(size 1.27 1.27)
+				)
+			)
+		)
+		(property "JLCPCB Part #" "C2909336"
+			(at 179.07 101.6 90)
+			(hide yes)
+			(show_name no)
+			(do_not_autoplace no)
+			(effects
+				(font
+					(size 1.27 1.27)
+				)
+			)
+		)
+		(property "Distributor Link" "https://www.lcsc.com/product-detail/C2909336.html"
 			(at 179.07 101.6 90)
 			(hide yes)
@@
 			)
 		)
-		(property "Distributor Link" "https://www.lcsc.com/product-detail/C60474.html?s_z=s_p_CC0402KRX7R7BB104&spm=wm.fly.bg.0.xh&lcsc_vid=RlRYUFFURFcNVFIDFVMMXgZSRlJeUABSQVNfAwJfQwIxVlNeTldcUFdQQFNXVTsOAxUeFF5JWBYZEEoKFBINSQcJGk4NBhADEA4cHktXRlVcSQwSGg0%3D"
-			(at 127 90.17 0)
-			(hide yes)
-			(show_name no)
-			(do_not_autoplace no)
-			(effects
-				(font
-					(size 1.27 1.27)
-				)
-			)
-		)
 		(property "Manufacturer" "YAGEO"
 			(at 127 90.17 0)
@@
 		)
 		(property "MPN" "CC0402KRX7R7BB104"
+			(at 127 90.17 0)
+			(hide yes)
+			(show_name no)
+			(do_not_autoplace no)
+			(effects
+				(font
+					(size 1.27 1.27)
+				)
+			)
+		)
+		(property "JLCPCB Part #" "C60474"
+			(at 127 90.17 0)
+			(hide yes)
+			(show_name no)
+			(do_not_autoplace no)
+			(effects
+				(font
+					(size 1.27 1.27)
+				)
+			)
+		)
+		(property "Distributor Link" "https://www.lcsc.com/product-detail/C60474.html"
 			(at 127 90.17 0)
 			(hide yes)
@@
 			)
 		)
-		(property "Distributor Link" "https://www.lcsc.com/product-detail/C157926.html?s_z=s_p_S4B-PH-K-S%28LF%29%28SN%29"
-			(at 109.22 101.6 0)
-			(hide yes)
-			(show_name no)
-			(do_not_autoplace no)
-			(effects
-				(font
-					(size 1.27 1.27)
-				)
-			)
-		)
 		(property "MPN" "S4B-PH-K-S(LF)(SN)"
 			(at 109.22 101.6 0)
@@
 		)
 		(property "Manufacturer" "JST"
+			(at 109.22 101.6 0)
+			(hide yes)
+			(show_name no)
+			(do_not_autoplace no)
+			(effects
+				(font
+					(size 1.27 1.27)
+				)
+			)
+		)
+		(property "JLCPCB Part #" "C157926"
+			(at 109.22 101.6 0)
+			(hide yes)
+			(show_name no)
+			(do_not_autoplace no)
+			(effects
+				(font
+					(size 1.27 1.27)
+				)
+			)
+		)
+		(property "Distributor Link" "https://www.lcsc.com/product-detail/C157926.html"
 			(at 109.22 101.6 0)
 			(hide yes)
@@
 			)
 		)
+		(property "Manufacturer" "FOJAN"
+			(at 179.07 104.14 90)
+			(hide yes)
+			(show_name no)
+			(do_not_autoplace no)
+			(effects
+				(font
+					(size 1.27 1.27)
+				)
+			)
+		)
+		(property "Distributor" "LCSC"
+			(at 179.07 104.14 90)
+			(hide yes)
+			(show_name no)
+			(do_not_autoplace no)
+			(effects
+				(font
+					(size 1.27 1.27)
+				)
+			)
+		)
+		(property "MPN" "FRC0402F2200TS"
+			(at 179.07 104.14 90)
+			(hide yes)
+			(show_name no)
+			(do_not_autoplace no)
+			(effects
+				(font
+					(size 1.27 1.27)
+				)
+			)
+		)
+		(property "JLCPCB Part #" "C2909336"
+			(at 179.07 104.14 90)
+			(hide yes)
+			(show_name no)
+			(do_not_autoplace no)
+			(effects
+				(font
+					(size 1.27 1.27)
+				)
+			)
+		)
 		(property "Distributor Link" "https://www.lcsc.com/product-detail/C2909336.html"
 			(at 179.07 104.14 90)
 			(hide yes)
-			(show_name no)
-			(do_not_autoplace no)
-			(effects
-				(font
-					(size 1.27 1.27)
-				)
-			)
-		)
-		(property "Manufacturer" "FOJAN"
-			(at 179.07 104.14 90)
-			(hide yes)
-			(show_name no)
-			(do_not_autoplace no)
-			(effects
-				(font
-					(size 1.27 1.27)
-				)
-			)
-		)
-		(property "Distributor" "LCSC"
-			(at 179.07 104.14 90)
-			(hide yes)
-			(show_name no)
-			(do_not_autoplace no)
-			(effects
-				(font
-					(size 1.27 1.27)
-				)
-			)
-		)
-		(property "MPN" "FRC0402F2200TS"
-			(at 179.07 104.14 90)
-			(hide yes)
