File: kicad/ldo.kicad_sch (KiCad schematic)
At the start: 5 parts, among them U3 MIC5365-3.3YD5

Commit message: fix(schematic): misc. fixes and stuff - sort all sheets - add the author's name to all sheets and update the date - add 0R resistor to the input of each crystal oscillator - reannotate all symbols - remove todo.md
Parts:
- renumbered D2 to D3, R8 to R7, U3 to U1
Changed lines of the file:
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@@
 	(paper "A4")
 	(title_block
-		(date "2026-05-27")
+		(date "2026-06-30")
 		(rev "1.0")
+		(comment 3 "Author: Odai J.")
 		(comment 4 "GitHub: https://github.com/odaij/stm32-bt-board")
 	)
@@
 		(dnp no)
 		(fields_autoplaced yes)
-		(property "Reference" "#PWR030"
+		(property "Reference" "#PWR023"
 			(at 142.24 123.19 0)
 			(hide yes)
@@
 			(project "stm32-bt-board"
 				(path "/9ab97115-0b3b-4897-8d44-f79e27c270d1/5ee7caa4-bcee-4f11-b707-877fa3e5f3cb"
-					(reference "#PWR030")
+					(reference "#PWR023")
 					(unit 1)
 				)
@@
 		(dnp no)
 		(fields_autoplaced yes)
-		(property "Reference" "U3"
+		(property "Reference" "U1"
 			(at 142.24 82.55 0)
 			(show_name no)
@@
 			(project "stm32-bt-board"
 				(path "/9ab97115-0b3b-4897-8d44-f79e27c270d1/5ee7caa4-bcee-4f11-b707-877fa3e5f3cb"
-					(reference "U3")
+					(reference "U1")
 					(unit 1)
 				)
@@
 		(dnp no)
 		(fields_autoplaced yes)
-		(property "Reference" "#PWR032"
+		(property "Reference" "#PWR022"
 			(at 123.19 123.19 0)
 			(hide yes)
@@
 			(project "stm32-bt-board"
 				(path "/9ab97115-0b3b-4897-8d44-f79e27c270d1/5ee7caa4-bcee-4f11-b707-877fa3e5f3cb"
-					(reference "#PWR032")
+					(reference "#PWR022")
 					(unit 1)
 				)
@@
 		(dnp no)
 		(fields_autoplaced yes)
-		(property "Reference" "R8"
+		(property "Reference" "R7"
 			(at 175.26 110.4899 0)
 			(show_name no)
@@
 			(project "stm32-bt-board"
 				(path "/9ab97115-0b3b-4897-8d44-f79e27c270d1/5ee7caa4-bcee-4f11-b707-877fa3e5f3cb"
-					(reference "R8")
+					(reference "R7")
 					(unit 1)
 				)
@@
 		(dnp no)
 		(fields_autoplaced yes)
-		(property "Reference" "#PWR031"
+		(property "Reference" "#PWR024"
 			(at 161.29 123.19 0)
 			(hide yes)
@@
 			(project "stm32-bt-board"
 				(path "/9ab97115-0b3b-4897-8d44-f79e27c270d1/5ee7caa4-bcee-4f11-b707-877fa3e5f3cb"
-					(reference "#PWR031")
+					(reference "#PWR024")
 					(unit 1)
 				)
@@
 		(dnp no)
 		(fields_autoplaced yes)
-		(property "Reference" "#PWR039"
+		(property "Reference" "#PWR021"
 			(at 177.8 91.44 0)
 			(hide yes)
@@
 			(project "stm32-bt-board"
 				(path "/9ab97115-0b3b-4897-8d44-f79e27c270d1/5ee7caa4-bcee-4f11-b707-877fa3e5f3cb"
-					(reference "#PWR039")
+					(reference "#PWR021")
 					(unit 1)
 				)
@@
 		(dnp no)
 		(fields_autoplaced yes)
-		(property "Reference" "D2"
+		(property "Reference" "D3"
 			(at 176.53 95.5674 90)
 			(show_name no)
@@
 			(project "stm32-bt-board"
 				(path "/9ab97115-0b3b-4897-8d44-f79e27c270d1/5ee7caa4-bcee-4f11-b707-877fa3e5f3cb"
-					(reference "D2")
+					(reference "D3")
 					(unit 1)
 				)
@@
 		(dnp no)
 		(fields_autoplaced yes)
-		(property "Reference" "#PWR027"
+		(property "Reference" "#PWR020"
 			(at 115.57 91.44 0)
 			(hide yes)
@@
 			(project "stm32-bt-board"
 				(path "/9ab97115-0b3b-4897-8d44-f79e27c270d1/5ee7caa4-bcee-4f11-b707-877fa3e5f3cb"
-					(reference "#PWR027")
+					(reference "#PWR020")
 					(unit 1)
 				)
@@
 		(dnp no)
 		(fields_autoplaced yes)
-		(property "Reference" "#PWR041"
+		(property "Reference" "#PWR025"
 			(at 172.72 123.19 0)
 			(hide yes)
@@
 			(project "stm32-bt-board"
 				(path "/9ab97115-0b3b-4897-8d44-f79e27c270d1/5ee7caa4-bcee-4f11-b707-877fa3e5f3cb"
-					(reference "#PWR041")
+					(reference "#PWR025")
 					(unit 1)
 				)

Commit message: everything: select real components, refactor schematic, add a user-led driving circuit, and more
Parts:
- C18, C19: footprint (none) -> Capacitor_SMD:C_0603_1608Metric; Distributor (none) -> LCSC; Distributor Link (none) -> https://www.lcsc.com/product-detail/C307467.html?spm=wm.fly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; MPN (none) -> CL10A475KL8NRNC; Manufacturer (none) -> Samsung Electro-Mechanics
- D3: footprint (none) -> LED_SMD:LED_0402_1005Metric; Distributor (none) -> LCSC; Distributor Link (none) -> https://www.lcsc.com/product-detail/C511370.html?spm=wm.fly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; MPN (none) -> VLMS1500-GS08; Manufacturer (none) -> VISHAY
- R7: footprint (none) -> Resistor_SMD:R_0402_1005Metric
- U1: Distributor (none) -> LCSC; Distributor Link (none) -> https://www.lcsc.com/product-detail/C626098.html?s_z=n_q_MI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; MPN (none) -> MIC5365-3.3YD5-TR; Manufacturer (none) -> MICROCHIP
Changed lines of the file:
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@@
 			)
 		)
-		(property "Distributor Link" ""
+		(property "Distributor Link" "https://www.lcsc.com/product-detail/C626098.html?s_z=n_q_MIC5365-3.3YD5&spm=wm.fly.bg.0.xh&lcsc_vid=RlRYUFFURFcNVFIDFVMMXgZSRlJeUABSQVNfAwJfQwIxVlNeTldcXlNTQFVfUTsOAxUeFF5JWBYZEEoKFBINSQcJGk4%3D"
 			(at 142.24 92.71 0)
 			(hide yes)
@@
 			)
 		)
-		(property "Manufacturer" ""
+		(property "Manufacturer" "MICROCHIP"
 			(at 142.24 92.71 0)
 			(hide yes)
@@
 			)
 		)
-		(property "Manufacturer Part Number" ""
+		(property "Distributor" "LCSC"
+			(at 142.24 92.71 0)
+			(hide yes)
+			(show_name no)
+			(do_not_autoplace no)
+			(effects
+				(font
+					(size 1.27 1.27)
+				)
+			)
+		)
+		(property "MPN" "MIC5365-3.3YD5-TR"
 			(at 142.24 92.71 0)
 			(hide yes)
@@
 			)
 		)
-		(property "Footprint" ""
+		(property "Footprint" "Capacitor_SMD:C_0603_1608Metric"
 			(at 160.3248 105.41 0)
 			(hide yes)
@@
 			)
 		)
-		(property "Datasheet" ""
+		(property "Datasheet" "https://www.lcsc.com/datasheet/C307467.pdf?spm=wm.sxq.inf.ggs___wm.fly.bg.5.xh&lcsc_vid=RlRYUFFURFcNVFIDFVMMXgZSRlJeUABSQVNfAwJfQwIxVlNeTldcX1VVRFlfUDsOAxUeFF5JWBYZEEoKFBINSQcJGk4eFQsCAgIaSgADAwAHC0slRlNdUVVXWQkaCgg%3D"
 			(at 161.29 101.6 0)
 			(hide yes)
@@
 			)
 		)
-		(property "Description" "Unpolarized capacitor"
+		(property "Description" "CAP CER 4.7uF 35V X5R 0603"
 			(at 161.29 101.6 0)
 			(hide yes)
@@
 			)
 		)
-		(property "Distributor Link" ""
+		(property "Distributor Link" "https://www.lcsc.com/product-detail/C307467.html?spm=wm.fly.bg.5.xh&lcsc_vid=RlRYUFFURFcNVFIDFVMMXgZSRlJeUABSQVNfAwJfQwIxVlNeTldcX1VVRFlfUDsOAxUeFF5JWBYZEEoKFBINSQcJGk4eFQsCAgIaSgADAwAHC0slRlNdUVVXWQkaCgg%3D"
 			(at 161.29 101.6 0)
 			(hide yes)
@@
 			)
 		)
-		(property "Manufacturer" ""
+		(property "Manufacturer" "Samsung Electro-Mechanics"
 			(at 161.29 101.6 0)
 			(hide yes)
@@
 			)
 		)
-		(property "Manufacturer Part Number" ""
+		(property "Distributor" "LCSC"
+			(at 161.29 101.6 0)
+			(hide yes)
+			(show_name no)
+			(do_not_autoplace no)
+			(effects
+				(font
+					(size 1.27 1.27)
+				)
+			)
+		)
+		(property "MPN" "CL10A475KL8NRNC"
 			(at 161.29 101.6 0)
 			(hide yes)
@@
 			)
 		)
-		(property "Footprint" ""
+		(property "Footprint" "Capacitor_SMD:C_0603_1608Metric"
 			(at 124.1552 105.41 0)
 			(hide yes)
@@
 			)
 		)
-		(property "Datasheet" ""
+		(property "Datasheet" "https://www.lcsc.com/datasheet/C307467.pdf?spm=wm.sxq.inf.ggs___wm.fly.bg.5.xh&lcsc_vid=RlRYUFFURFcNVFIDFVMMXgZSRlJeUABSQVNfAwJfQwIxVlNeTldcX1VVRFlfUDsOAxUeFF5JWBYZEEoKFBINSQcJGk4eFQsCAgIaSgADAwAHC0slRlNdUVVXWQkaCgg%3D"
 			(at 123.19 101.6 0)
 			(hide yes)
@@
 			)
 		)
-		(property "Description" "Unpolarized capacitor"
+		(property "Description" "CAP CER 4.7uF 35V X5R 0603"
 			(at 123.19 101.6 0)
 			(hide yes)
@@
 			)
 		)
-		(property "Distributor Link" ""
+		(property "Distributor Link" "https://www.lcsc.com/product-detail/C307467.html?spm=wm.fly.bg.5.xh&lcsc_vid=RlRYUFFURFcNVFIDFVMMXgZSRlJeUABSQVNfAwJfQwIxVlNeTldcX1VVRFlfUDsOAxUeFF5JWBYZEEoKFBINSQcJGk4eFQsCAgIaSgADAwAHC0slRlNdUVVXWQkaCgg%3D"
 			(at 123.19 101.6 0)
 			(hide yes)
@@
 			)
 		)
-		(property "Manufacturer" ""
+		(property "Manufacturer" "Samsung Electro-Mechanics"
 			(at 123.19 101.6 0)
 			(hide yes)
@@
 			)
 		)
-		(property "Manufacturer Part Number" ""
+		(property "Distributor" "LCSC"
+			(at 123.19 101.6 0)
+			(hide yes)
+			(show_name no)
+			(do_not_autoplace no)
+			(effects
+				(font
+					(size 1.27 1.27)
+				)
+			)
+		)
+		(property "MPN" "CL10A475KL8NRNC"
 			(at 123.19 101.6 0)
 			(hide yes)
@@
 			)
 		)
-		(property "Footprint" ""
+		(property "Footprint" "Resistor_SMD:R_0402_1005Metric"
 			(at 170.942 111.76 90)
 			(hide yes)
@@
 			)
 		)
-		(property "Manufacturer Part Number" ""
+		(property "Distributor" ""
 			(at 172.72 111.76 0)
 			(hide yes)
@@
 			)
 		)
-		(property "Footprint" ""
+		(property "Footprint" "LED_SMD:LED_0402_1005Metric"
 			(at 172.72 95.25 0)
 			(hide yes)
@@
 			)
 		)
-		(property "Datasheet" ""
+		(property "Datasheet" "https://www.lcsc.com/datasheet/C511370.pdf?spm=wm.sxq.inf.ggs___wm.fly.bg.11.xh&lcsc_vid=RlRYUFFURFcNVFIDFVMMXgZSRlJeUABSQVNfAwJfQwIxVlNeTlddVFRWQVdYUTsOAxUeFF5JWBYZEEoKFBINSQcJGk4NBhADEA4cHktSRlNADxALGw%3D%3D"
 			(at 172.72 95.25 0)
 			(hide yes)
@@
 			)
 		)
-		(property "Description" "Light emitting diode"
+		(property "Description" "LED RED 0402 SMD"
 			(at 172.72 95.25 0)
 			(hide yes)
@@
 			)
 		)
-		(property "Distributor Link" ""
+		(property "Distributor Link" "https://www.lcsc.com/product-detail/C511370.html?spm=wm.fly.bg.11.xh&lcsc_vid=RlRYUFFURFcNVFIDFVMMXgZSRlJeUABSQVNfAwJfQwIxVlNeTlddVFRWQVdYUTsOAxUeFF5JWBYZEEoKFBINSQcJGk4NBhADEA4cHktSRlNADxALGw%3D%3D"
 			(at 172.72 95.25 90)
 			(hide yes)
@@
 			)
 		)
-		(property "Manufacturer" ""
+		(property "Manufacturer" "VISHAY"
 			(at 172.72 95.25 90)
 			(hide yes)
@@
 			)
 		)
-		(property "Manufacturer Part Number" ""
+		(property "Distributor" "LCSC"
 			(at 172.72 95.25 90)
 			(hide yes)
+			(show_name no)
+			(do_not_autoplace no)
+			(effects
+				(font
+					(size 1.27 1.27)
+				)
+			)
+		)
+		(property "MPN" "VLMS1500-GS08"
+			(at 172.72 95.25 90)
+			(hide yes)

Commit message: feat(components): add details
Parts:
- D3: value LED -> VLMS1500-GS08
Changed lines of the file:
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@@
 			)
 		)
-		(property "Value" "LED"
+		(property "Value" "VLMS1500-GS08"
 			(at 176.53 98.1074 90)
 			(show_name no)

Commit message: feat(BOM): fill missing parts in BOM
Parts:
- R7: Distributor (none) -> LCSC; Distributor Link (none) -> https://www.lcsc.com/product-detail/C2909336.html; MPN (none) -> FRC0402F2200TS; Manufacturer (none) -> FOJAN
Changed lines of the file:
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@@
 			)
 		)
-		(property "Datasheet" ""
+		(property "Datasheet" "https://www.lcsc.com/datasheet/C2909336.pdf"
 			(at 172.72 111.76 0)
 			(hide yes)
@@
 			)
 		)
-		(property "Description" "Resistor"
+		(property "Description" "RES 220Ω ±1% 62.5mW 0402"
 			(at 172.72 111.76 0)
 			(hide yes)
@@
 			)
 		)
-		(property "Distributor Link" ""
+		(property "Distributor Link" "https://www.lcsc.com/product-detail/C2909336.html"
 			(at 172.72 111.76 0)
 			(hide yes)
@@
 			)
 		)
-		(property "Manufacturer" ""
+		(property "Manufacturer" "FOJAN"
 			(at 172.72 111.76 0)
 			(hide yes)
@@
 			)
 		)
-		(property "Distributor" ""
+		(property "Distributor" "LCSC"
 			(at 172.72 111.76 0)
 			(hide yes)
+			(show_name no)
+			(do_not_autoplace no)
+			(effects
+				(font
+					(size 1.27 1.27)
+				)
+			)
+		)
+		(property "MPN" "FRC0402F2200TS"
+			(at 172.72 111.76 0)
+			(hide yes)

Commit message: feat(manuf.): edit BOM and CPL to match JLCPCB's requirements
however, please pay close attention to the rotations during ordering, especially for the SOT components, as JLCPCB messes them up a bit, same for the connector and the filter
Parts:
- C18, C19: Distributor Link https://www.lcsc.com/product-detail/C307467.html?spm=wm.fly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 -> https://www.lcsc.com/product-detail/C307467.html; JLCPCB Part # (none) -> C307467
- D3: Distributor Link https://www.lcsc.com/product-detail/C511370.html?spm=wm.fly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 -> https://www.lcsc.com/product-detail/C511370.html; JLCPCB Part # (none) -> C511370
- R7: JLCPCB Part # (none) -> C2909336
- U1: Distributor Link https://www.lcsc.com/product-detail/C626098.html?s_z=n_q_MI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 -> https://www.lcsc.com/product-detail/C626098.html; JLCPCB Part # (none) -> C626098
Changed lines of the file:
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@@
-			)
-		)
-		(property "Distributor Link" "https://www.lcsc.com/product-detail/C626098.html?s_z=n_q_MIC5365-3.3YD5&spm=wm.fly.bg.0.xh&lcsc_vid=RlRYUFFURFcNVFIDFVMMXgZSRlJeUABSQVNfAwJfQwIxVlNeTldcXlNTQFVfUTsOAxUeFF5JWBYZEEoKFBINSQcJGk4%3D"
-			(at 142.24 92.71 0)
-			(hide yes)
-			(show_name no)
-			(do_not_autoplace no)
-			(effects
-				(font
-					(size 1.27 1.27)
-				)
 			)
 		)
@@
 		)
 		(property "MPN" "MIC5365-3.3YD5-TR"
+			(at 142.24 92.71 0)
+			(hide yes)
+			(show_name no)
+			(do_not_autoplace no)
+			(effects
+				(font
+					(size 1.27 1.27)
+				)
+			)
+		)
+		(property "JLCPCB Part #" "C626098"
+			(at 142.24 92.71 0)
+			(hide yes)
+			(show_name no)
+			(do_not_autoplace no)
+			(effects
+				(font
+					(size 1.27 1.27)
+				)
+			)
+		)
+		(property "Distributor Link" "https://www.lcsc.com/product-detail/C626098.html"
 			(at 142.24 92.71 0)
 			(hide yes)
@@
 			)
 		)
-		(property "Distributor Link" "https://www.lcsc.com/product-detail/C307467.html?spm=wm.fly.bg.5.xh&lcsc_vid=RlRYUFFURFcNVFIDFVMMXgZSRlJeUABSQVNfAwJfQwIxVlNeTldcX1VVRFlfUDsOAxUeFF5JWBYZEEoKFBINSQcJGk4eFQsCAgIaSgADAwAHC0slRlNdUVVXWQkaCgg%3D"
-			(at 161.29 101.6 0)
-			(hide yes)
-			(show_name no)
-			(do_not_autoplace no)
-			(effects
-				(font
-					(size 1.27 1.27)
-				)
-			)
-		)
 		(property "Manufacturer" "Samsung Electro-Mechanics"
 			(at 161.29 101.6 0)
@@
 		)
 		(property "MPN" "CL10A475KL8NRNC"
+			(at 161.29 101.6 0)
+			(hide yes)
+			(show_name no)
+			(do_not_autoplace no)
+			(effects
+				(font
+					(size 1.27 1.27)
+				)
+			)
+		)
+		(property "JLCPCB Part #" "C307467"
+			(at 161.29 101.6 0)
+			(hide yes)
+			(show_name no)
+			(do_not_autoplace no)
+			(effects
+				(font
+					(size 1.27 1.27)
+				)
+			)
+		)
+		(property "Distributor Link" "https://www.lcsc.com/product-detail/C307467.html"
 			(at 161.29 101.6 0)
 			(hide yes)
@@
 			)
 		)
-		(property "Distributor Link" "https://www.lcsc.com/product-detail/C307467.html?spm=wm.fly.bg.5.xh&lcsc_vid=RlRYUFFURFcNVFIDFVMMXgZSRlJeUABSQVNfAwJfQwIxVlNeTldcX1VVRFlfUDsOAxUeFF5JWBYZEEoKFBINSQcJGk4eFQsCAgIaSgADAwAHC0slRlNdUVVXWQkaCgg%3D"
-			(at 123.19 101.6 0)
-			(hide yes)
-			(show_name no)
-			(do_not_autoplace no)
-			(effects
-				(font
-					(size 1.27 1.27)
-				)
-			)
-		)
 		(property "Manufacturer" "Samsung Electro-Mechanics"
 			(at 123.19 101.6 0)
@@
 		)
 		(property "MPN" "CL10A475KL8NRNC"
+			(at 123.19 101.6 0)
+			(hide yes)
+			(show_name no)
+			(do_not_autoplace no)
+			(effects
+				(font
+					(size 1.27 1.27)
+				)
+			)
+		)
+		(property "JLCPCB Part #" "C307467"
+			(at 123.19 101.6 0)
+			(hide yes)
+			(show_name no)
+			(do_not_autoplace no)
+			(effects
+				(font
+					(size 1.27 1.27)
+				)
+			)
+		)
+		(property "Distributor Link" "https://www.lcsc.com/product-detail/C307467.html"
 			(at 123.19 101.6 0)
 			(hide yes)
@@
 			)
 		)
-		(property "Distributor Link" "https://www.lcsc.com/product-detail/C2909336.html"
-			(at 172.72 111.76 0)
-			(hide yes)
-			(show_name no)
-			(do_not_autoplace no)
-			(effects
-				(font
-					(size 1.27 1.27)
-				)
-			)
-		)
 		(property "Manufacturer" "FOJAN"
 			(at 172.72 111.76 0)
@@
 		)
 		(property "MPN" "FRC0402F2200TS"
+			(at 172.72 111.76 0)
+			(hide yes)
+			(show_name no)
+			(do_not_autoplace no)
+			(effects
+				(font
+					(size 1.27 1.27)
+				)
+			)
+		)
+		(property "JLCPCB Part #" "C2909336"
+			(at 172.72 111.76 0)
+			(hide yes)
+			(show_name no)
+			(do_not_autoplace no)
+			(effects
+				(font
+					(size 1.27 1.27)
+				)
+			)
+		)
+		(property "Distributor Link" "https://www.lcsc.com/product-detail/C2909336.html"
 			(at 172.72 111.76 0)
 			(hide yes)
@@
 			)
 		)
-		(property "Distributor Link" "https://www.lcsc.com/product-detail/C511370.html?spm=wm.fly.bg.11.xh&lcsc_vid=RlRYUFFURFcNVFIDFVMMXgZSRlJeUABSQVNfAwJfQwIxVlNeTlddVFRWQVdYUTsOAxUeFF5JWBYZEEoKFBINSQcJGk4NBhADEA4cHktSRlNADxALGw%3D%3D"
-			(at 172.72 95.25 90)
-			(hide yes)
-			(show_name no)
-			(do_not_autoplace no)
-			(effects
-				(font
-					(size 1.27 1.27)
-				)
-			)
-		)
 		(property "Manufacturer" "VISHAY"
 			(at 172.72 95.25 90)
@@
 			(at 172.72 95.25 90)
 			(hide yes)
+			(show_name no)
+			(do_not_autoplace no)
+			(effects
+				(font
+					(size 1.27 1.27)
+				)
+			)
+		)
+		(property "JLCPCB Part #" "C511370"
+			(at 172.72 95.25 90)
+			(hide yes)
+			(show_name no)
+			(do_not_autoplace no)
+			(effects
+				(font
+					(size 1.27 1.27)
+				)
+			)
+		)
+		(property "Distributor Link" "https://www.lcsc.com/product-detail/C511370.html"
+			(at 172.72 95.25 90)
+			(hide yes)
