File: kicad/mcu.kicad_sch (KiCad schematic)
At the start: 1 part, among them U1 STM32WB55CEU6

Commit message: fix(schematic): misc. fixes and stuff - sort all sheets - add the author's name to all sheets and update the date - add 0R resistor to the input of each crystal oscillator - reannotate all symbols - remove todo.md
Parts:
- renumbered U1 to U4
Changed lines of the file:
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@@
 	(paper "A4")
 	(title_block
-		(date "2026-05-27")
+		(date "2026-06-30")
 		(rev "1.0")
+		(comment 3 "Author: Odai J.")
 		(comment 4 "GitHub: https://github.com/odaij/stm32-bt-board")
 	)
@@
 		(dnp no)
 		(fields_autoplaced yes)
-		(property "Reference" "#PWR010"
+		(property "Reference" "#PWR01"
 			(at 140.97 71.12 0)
 			(hide yes)
@@
 			(project "stm32-bt-board"
 				(path "/9ab97115-0b3b-4897-8d44-f79e27c270d1/647642cc-3894-4f8c-9e36-c4f1abaf1fd9"
-					(reference "#PWR010")
+					(reference "#PWR01")
 					(unit 1)
 				)
@@
 		(in_pos_files yes)
 		(dnp no)
-		(property "Reference" "U1"
+		(property "Reference" "U4"
 			(at 171.704 76.2 0)
 			(show_name no)
@@
 			(project "stm32-bt-board"
 				(path "/9ab97115-0b3b-4897-8d44-f79e27c270d1/647642cc-3894-4f8c-9e36-c4f1abaf1fd9"
-					(reference "U1")
+					(reference "U4")
 					(unit 1)
 				)
@@
 		(dnp no)
 		(fields_autoplaced yes)
-		(property "Reference" "#PWR01"
+		(property "Reference" "#PWR02"
 			(at 148.59 165.1 0)
 			(hide yes)
@@
 			(project "stm32-bt-board"
 				(path "/9ab97115-0b3b-4897-8d44-f79e27c270d1/647642cc-3894-4f8c-9e36-c4f1abaf1fd9"
-					(reference "#PWR01")
+					(reference "#PWR02")
 					(unit 1)
 				)
@@
 			(project "stm32-bt-board"
 				(path "/9ab97115-0b3b-4897-8d44-f79e27c270d1/647642cc-3894-4f8c-9e36-c4f1abaf1fd9"
-					(page "7")
+					(page "4")
 				)
 			)
@@
 			(project "stm32-bt-board"
 				(path "/9ab97115-0b3b-4897-8d44-f79e27c270d1/647642cc-3894-4f8c-9e36-c4f1abaf1fd9"
-					(page "9")
+					(page "3")
 				)
 			)
@@
 			(project "stm32-bt-board"
 				(path "/9ab97115-0b3b-4897-8d44-f79e27c270d1/647642cc-3894-4f8c-9e36-c4f1abaf1fd9"
-					(page "8")
+					(page "6")
 				)
 			)
@@
 			(project "stm32-bt-board"
 				(path "/9ab97115-0b3b-4897-8d44-f79e27c270d1/647642cc-3894-4f8c-9e36-c4f1abaf1fd9"
-					(page "5")
+					(page "7")
 				)
 			)
@@
 			(project "stm32-bt-board"
 				(path "/9ab97115-0b3b-4897-8d44-f79e27c270d1/647642cc-3894-4f8c-9e36-c4f1abaf1fd9"
-					(page "6")
-				)
-			)
+					(page "5")
+				)
+			)

Commit message: everything: select real components, refactor schematic, add a user-led driving circuit, and more
Parts:
- U4: Distributor (none) -> Mouser; Distributor Link (none) -> https://mou.sr/4AjC6F3; MPN (none) -> STM32WB55CEU6; Manufacturer (none) -> ST
Changed lines of the file:
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@@
 			)
 		)
-		(property "Distributor Link" ""
+		(property "Distributor Link" "https://mou.sr/4AjC6F3"
 			(at 151.13 115.57 0)
 			(hide yes)
@@
 			)
 		)
-		(property "Manufacturer" ""
+		(property "Manufacturer" "ST"
 			(at 151.13 115.57 0)
 			(hide yes)
@@
 			)
 		)
-		(property "Manufacturer Part Number" ""
+		(property "Distributor" "Mouser"
 			(at 151.13 115.57 0)
 			(hide yes)
+			(show_name no)
+			(do_not_autoplace no)
+			(effects
+				(font
+					(size 1.27 1.27)
+				)
+			)
+		)
+		(property "MPN" "STM32WB55CEU6"
+			(at 151.13 115.57 0)
+			(hide yes)

Commit message: feat(BOM): fill missing parts in BOM
Parts:
- U4: Distributor Mouser -> LCSC; Distributor Link https://mou.sr/4AjC6F3 -> https://www.lcsc.com/product-detail/C911135.html?s_z=s_p_ST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
Changed lines of the file:
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@@
 			)
 		)
-		(property "Distributor Link" "https://mou.sr/4AjC6F3"
+		(property "Distributor Link" "https://www.lcsc.com/product-detail/C911135.html?s_z=s_p_STM32WB55CEU6"
 			(at 151.13 115.57 0)
 			(hide yes)
@@
 			)
 		)
-		(property "Distributor" "Mouser"
+		(property "Distributor" "LCSC"
 			(at 151.13 115.57 0)
 			(hide yes)

Commit message: feat(manuf.): edit BOM and CPL to match JLCPCB's requirements
however, please pay close attention to the rotations during ordering, especially for the SOT components, as JLCPCB messes them up a bit, same for the connector and the filter
Parts:
- U4: Distributor Link https://www.lcsc.com/product-detail/C911135.html?s_z=s_p_ST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 -> https://www.lcsc.com/product-detail/C911135.html; JLCPCB Part # (none) -> C911135
Changed lines of the file:
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@@
-			)
-		)
-		(property "Distributor Link" "https://www.lcsc.com/product-detail/C911135.html?s_z=s_p_STM32WB55CEU6"
-			(at 151.13 115.57 0)
-			(hide yes)
-			(show_name no)
-			(do_not_autoplace no)
-			(effects
-				(font
-					(size 1.27 1.27)
-				)
 			)
 		)
@@
 			(at 151.13 115.57 0)
 			(hide yes)
+			(show_name no)
+			(do_not_autoplace no)
+			(effects
+				(font
+					(size 1.27 1.27)
+				)
+			)
+		)
+		(property "JLCPCB Part #" "C911135"
+			(at 151.13 115.57 0)
+			(hide yes)
+			(show_name no)
+			(do_not_autoplace no)
+			(effects
+				(font
+					(size 1.27 1.27)
+				)
+			)
+		)
+		(property "Distributor Link" "https://www.lcsc.com/product-detail/C911135.html"
+			(at 151.13 115.57 0)
+			(hide yes)
