File: kicad/mcu_rf.kicad_sch (KiCad schematic)
At the start: 5 parts, among them J1 Conn_Coaxial

Commit message: fix(schematic): misc. fixes and stuff - sort all sheets - add the author's name to all sheets and update the date - add 0R resistor to the input of each crystal oscillator - reannotate all symbols - remove todo.md
Parts:
- renumbered C14 to C12, C15 to C13
Other:
- moved on the sheet: FL1, J1
Changed lines of the file:
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@@
 	(paper "A4")
 	(title_block
-		(date "2026-05-27")
+		(date "2026-06-30")
 		(rev "1.0")
+		(comment 3 "Author: Odai J.")
 		(comment 4 "GitHub: https://github.com/odaij/stm32-bt-board")
 	)
 	(rectangle
 		(start 88.9 76.2)
-		(end 194.31 118.11)
+		(end 198.12 118.11)
 		(stroke
 			(width 0)
@@
 	)
 	(junction
-		(at 151.13 104.14)
+		(at 124.46 93.98)
+		(diameter 0)
+		(color 0 0 0 0)
+	)
+	(junction
+		(at 156.21 104.14)
 		(diameter 0)
 		(color 0 0 0 0)
@@
 		(color 0 0 0 0)
 	)
-	(junction
-		(at 124.46 93.98)
-		(diameter 0)
-		(color 0 0 0 0)
-	)
 	(wire
 		(pts
@@
 	(wire
 		(pts
-			(xy 151.13 100.33) (xy 151.13 104.14)
+			(xy 156.21 100.33) (xy 156.21 104.14)
 		)
 		(stroke
@@
 	(wire
 		(pts
-			(xy 148.59 100.33) (xy 148.59 104.14)
+			(xy 153.67 100.33) (xy 153.67 104.14)
 		)
 		(stroke
@@
 	(wire
 		(pts
-			(xy 151.13 104.14) (xy 151.13 107.95)
+			(xy 156.21 104.14) (xy 156.21 107.95)
 		)
 		(stroke
@@
 	(wire
 		(pts
-			(xy 160.02 93.98) (xy 170.18 93.98)
+			(xy 165.1 93.98) (xy 175.26 93.98)
 		)
 		(stroke
@@
 	(wire
 		(pts
-			(xy 148.59 104.14) (xy 151.13 104.14)
+			(xy 153.67 104.14) (xy 156.21 104.14)
 		)
 		(stroke
@@
 	(wire
 		(pts
-			(xy 175.26 99.06) (xy 175.26 107.95)
+			(xy 180.34 99.06) (xy 180.34 107.95)
 		)
 		(stroke
@@
 	(wire
 		(pts
-			(xy 124.46 93.98) (xy 139.7 93.98)
+			(xy 124.46 93.98) (xy 144.78 93.98)
 		)
 		(stroke
@@
 	)
 	(label "RF_ANT"
-		(at 162.56 93.98 0)
+		(at 167.64 93.98 0)
 		(effects
 			(font
@@
 		(effects
 			(font
-				(size 0.508 0.508)
+				(size 1.27 1.27)
 			)
 			(justify left bottom)
@@
 	(symbol
 		(lib_id "power:GND")
-		(at 175.26 107.95 0)
+		(at 180.34 107.95 0)
 		(unit 1)
 		(body_style 1)
@@
 		(dnp no)
 		(fields_autoplaced yes)
-		(property "Reference" "#PWR05"
-			(at 175.26 114.3 0)
+		(property "Reference" "#PWR07"
+			(at 180.34 114.3 0)
 			(hide yes)
 			(show_name no)
@@
 		)
 		(property "Value" "GND"
-			(at 175.26 113.03 0)
+			(at 180.34 113.03 0)
 			(hide yes)
 			(show_name no)
@@
 		)
 		(property "Footprint" ""
-			(at 175.26 107.95 0)
+			(at 180.34 107.95 0)
 			(hide yes)
 			(show_name no)
@@
 		)
 		(property "Datasheet" ""
-			(at 175.26 107.95 0)
+			(at 180.34 107.95 0)
 			(hide yes)
 			(show_name no)
@@
 		)
 		(property "Description" "Power symbol creates a global label with name \"GND\" , ground"
-			(at 175.26 107.95 0)
+			(at 180.34 107.95 0)
 			(hide yes)
 			(show_name no)
@@
 			(project "stm32-bt-board"
 				(path "/9ab97115-0b3b-4897-8d44-f79e27c270d1/647642cc-3894-4f8c-9e36-c4f1abaf1fd9/387be5c2-c06a-4ce1-b441-93a813b84222"
-					(reference "#PWR05")
+					(reference "#PWR07")
 					(unit 1)
 				)
@@
 		(dnp no)
 		(fields_autoplaced yes)
-		(property "Reference" "#PWR03"
+		(property "Reference" "#PWR05"
 			(at 124.46 114.3 0)
 			(hide yes)
@@
 			(project "stm32-bt-board"
 				(path "/9ab97115-0b3b-4897-8d44-f79e27c270d1/647642cc-3894-4f8c-9e36-c4f1abaf1fd9/387be5c2-c06a-4ce1-b441-93a813b84222"
-					(reference "#PWR03")
+					(reference "#PWR05")
 					(unit 1)
 				)
@@
 	(symbol
 		(lib_id "#odaij_RF_Filter:TDK_DLF162500LT-5028A1")
-		(at 149.86 93.98 0)
+		(at 154.94 93.98 0)
 		(unit 1)
 		(body_style 1)
@@
 		(fields_autoplaced yes)
 		(property "Reference" "FL1"
-			(at 149.86 85.09 0)
+			(at 154.94 85.09 0)
 			(show_name no)
 			(do_not_autoplace no)
@@
 		)
 		(property "Value" "TDK_DLF162500LT-5028A1"
-			(at 149.86 87.63 0)
+			(at 154.94 87.63 0)
 			(show_name no)
 			(do_not_autoplace no)
@@
 		)
 		(property "Footprint" "#odaij_RF_Filter:TDK_DLF162500LT-5028A1"
-			(at 149.86 93.98 0)
+			(at 154.94 93.98 0)
 			(hide yes)
 			(show_name no)
@@
 		)
 		(property "Datasheet" "https://product.tdk.com/en/system/files/dam/doc/product/rf/rf/filter/catalog/rf_lpf_dlf162500lt-5028a1_en.pdf"
-			(at 149.86 93.98 0)
+			(at 154.94 93.98 0)
 			(hide yes)
 			(show_name no)
@@
 		)
 		(property "Description" "Multilayer Low Pass Filter For 2400-2500MHz"
-			(at 149.86 93.98 0)
+			(at 154.94 93.98 0)
 			(hide yes)
 			(show_name no)
@@
 		)
 		(property "KLC_S3.3" ""
-			(at 149.86 93.98 0)
+			(at 154.94 93.98 0)
 			(hide yes)
 			(show_name no)
@@
 		)
 		(property "KLC_S4.1" ""
-			(at 149.86 93.98 0)
+			(at 154.94 93.98 0)
 			(hide yes)
 			(show_name no)
@@
 		)
 		(property "Distributor Link" ""
-			(at 149.86 93.98 0)
+			(at 154.94 93.98 0)
 			(hide yes)
 			(show_name no)
@@
 		)
 		(property "Manufacturer" ""
-			(at 149.86 93.98 0)
+			(at 154.94 93.98 0)
 			(hide yes)
 			(show_name no)
@@
 		)
 		(property "Manufacturer Part Number" ""
-			(at 149.86 93.98 0)
+			(at 154.94 93.98 0)
 			(hide yes)
 			(show_name no)
@@
 		(dnp no)
 		(fields_autoplaced yes)
-		(property "Reference" "#PWR02"
+		(property "Reference" "#PWR04"
 			(at 106.68 114.3 0)
 			(hide yes)
@@
 			(project "stm32-bt-board"
 				(path "/9ab97115-0b3b-4897-8d44-f79e27c270d1/647642cc-3894-4f8c-9e36-c4f1abaf1fd9/387be5c2-c06a-4ce1-b441-93a813b84222"
-					(reference "#PWR02")
+					(reference "#PWR04")
 					(unit 1)
 				)
@@
 		(dnp no)
 		(fields_autoplaced yes)
-		(property "Reference" "C14"
+		(property "Reference" "C12"
 			(at 110.49 96.5199 0)
 			(show_name no)
@@
 			(project "stm32-bt-board"
 				(path "/9ab97115-0b3b-4897-8d44-f79e27c270d1/647642cc-3894-4f8c-9e36-c4f1abaf1fd9/387be5c2-c06a-4ce1-b441-93a813b84222"
-					(reference "C14")
+					(reference "C12")
 					(unit 1)
 				)
@@
 	(symbol
 		(lib_id "power:GND")
-		(at 151.13 107.95 0)
+		(at 156.21 107.95 0)
 		(unit 1)
 		(body_style 1)
@@
 		(dnp no)
 		(fields_autoplaced yes)
-		(property "Reference" "#PWR04"
-			(at 151.13 114.3 0)
+		(property "Reference" "#PWR06"
+			(at 156.21 114.3 0)
 			(hide yes)
 			(show_name no)
@@
 		)
 		(property "Value" "GND"
-			(at 151.13 113.03 0)
+			(at 156.21 113.03 0)
 			(hide yes)
 			(show_name no)
@@
 		)
 		(property "Footprint" ""
-			(at 151.13 107.95 0)
+			(at 156.21 107.95 0)
 			(hide yes)
 			(show_name no)
@@
 		)
 		(property "Datasheet" ""
-			(at 151.13 107.95 0)
+			(at 156.21 107.95 0)
 			(hide yes)
 			(show_name no)
@@
 		)
 		(property "Description" "Power symbol creates a global label with name \"GND\" , ground"
-			(at 151.13 107.95 0)
+			(at 156.21 107.95 0)
 			(hide yes)
 			(show_name no)
@@
 			(project "stm32-bt-board"
 				(path "/9ab97115-0b3b-4897-8d44-f79e27c270d1/647642cc-3894-4f8c-9e36-c4f1abaf1fd9/387be5c2-c06a-4ce1-b441-93a813b84222"
-					(reference "#PWR04")
+					(reference "#PWR06")
 					(unit 1)
 				)
@@
 		(dnp no)
 		(fields_autoplaced yes)
-		(property "Reference" "C15"
+		(property "Reference" "C13"
 			(at 128.27 96.5199 0)
 			(show_name no)
@@
 			(project "stm32-bt-board"
 				(path "/9ab97115-0b3b-4897-8d44-f79e27c270d1/647642cc-3894-4f8c-9e36-c4f1abaf1fd9/387be5c2-c06a-4ce1-b441-93a813b84222"
-					(reference "C15")
+					(reference "C13")
 					(unit 1)
 				)
@@
 	(symbol
 		(lib_id "Connector:Conn_Coaxial")
-		(at 175.26 93.98 0)
+		(at 180.34 93.98 0)
 		(unit 1)
 		(body_style 1)
@@
 		(fields_autoplaced yes)
 		(property "Reference" "J1"
-			(at 179.07 93.0031 0)
+			(at 184.15 93.0031 0)
 			(show_name no)
 			(do_not_autoplace no)
@@
 		)
 		(property "Value" "Conn_Coaxial"
-			(at 179.07 95.5431 0)
+			(at 184.15 95.5431 0)
 			(show_name no)
 			(do_not_autoplace no)
@@
 		)
 		(property "Footprint" ""
-			(at 175.26 93.98 0)
+			(at 180.34 93.98 0)
 			(hide yes)
 			(show_name no)
@@
 		)
 		(property "Datasheet" ""
-			(at 175.26 93.98 0)
+			(at 180.34 93.98 0)
 			(hide yes)
 			(show_name no)
@@
 		)
 		(property "Description" "coaxial connector (BNC, SMA, SMB, SMC, Cinch/RCA, LEMO, ...)"
-			(at 175.26 93.98 0)
+			(at 180.34 93.98 0)
 			(hide yes)
 			(show_name no)
@@
 		)
 		(property "KLC_S3.3" ""
-			(at 175.26 93.98 0)
+			(at 180.34 93.98 0)
 			(hide yes)
 			(show_name no)
@@
 		)
 		(property "KLC_S4.1" ""
-			(at 175.26 93.98 0)
+			(at 180.34 93.98 0)
 			(hide yes)
 			(show_name no)
@@
 		)
 		(property "Distributor Link" ""
-			(at 175.26 93.98 0)
+			(at 180.34 93.98 0)
 			(hide yes)
 			(show_name no)
@@
 		)
 		(property "Manufacturer" ""
-			(at 175.26 93.98 0)
+			(at 180.34 93.98 0)
 			(hide yes)
 			(show_name no)
@@
 		)
 		(property "Manufacturer Part Number" ""
-			(at 175.26 93.98 0)
-			(hide yes)
-			(show_name no)
+			(at 180.34 93.98 0)
+			(hide yes)
+			(show_name no)

Commit message: everything: select real components, refactor schematic, add a user-led driving circuit, and more
Parts:
- C12: footprint (none) -> Capacitor_SMD:C_0402_1005Metric; Distributor (none) -> LCSC; MPN (none) -> GRM1555C1HR80BA01D; Manufacturer Part Number GRM1555C1HR80BA01D -> (none)
- C13: footprint (none) -> Capacitor_SMD:C_0402_1005Metric; Distributor (none) -> LCSC; MPN (none) -> GRM1555C1HR30WA01D; Manufacturer Part Number GRM1555C1HR30WA01D -> (none)
- FL1: Distributor (none) -> LCSC; Distributor Link (none) -> https://www.lcsc.com/product-detail/C531364.html?s_z=s_p_DL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; MPN (none) -> DLF162500LT-5028A1; Manufacturer (none) -> TDK
- L3: footprint (none) -> Inductor_SMD:L_0402_1005Metric; Distributor (none) -> LCSC; MPN (none) -> LQG15HS2N7S02D; Manufacturer Part Number LQG15HS2N7S02D -> (none)
Changed lines of the file:
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@@
 			)
 		)
-		(property "Distributor Link" ""
+		(property "Distributor Link" "https://www.lcsc.com/product-detail/C531364.html?s_z=s_p_DLF162500LT-5028A1&spm=wm.fly.bg.0.xh&lcsc_vid=RlRYUFFURFcNVFIDFVMMXgZSRlJeUABSQVNfAwJfQwIxVlNeTldcX1JQQVRbVjsOAxUeFF5JWBYZEEoKFBINSQcJGk4eFQsCAgIaSgADAwAHC0slRVldVVFfWQkaCgg%3D"
 			(at 154.94 93.98 0)
 			(hide yes)
@@
 			)
 		)
-		(property "Manufacturer" ""
+		(property "Manufacturer" "TDK"
 			(at 154.94 93.98 0)
 			(hide yes)
@@
 			)
 		)
-		(property "Manufacturer Part Number" ""
+		(property "Distributor" "LCSC"
+			(at 154.94 93.98 0)
+			(hide yes)
+			(show_name no)
+			(do_not_autoplace no)
+			(effects
+				(font
+					(size 1.27 1.27)
+				)
+			)
+		)
+		(property "MPN" "DLF162500LT-5028A1"
 			(at 154.94 93.98 0)
 			(hide yes)
@@
 			)
 		)
-		(property "Footprint" ""
+		(property "Footprint" "Capacitor_SMD:C_0402_1005Metric"
 			(at 107.6452 101.6 0)
 			(hide yes)
@@
 			)
 		)
-		(property "Datasheet" ""
+		(property "Datasheet" "https://www.lcsc.com/datasheet/C76988.pdf?spm=wm.sxq.inf.ggs___wm.fly.bg.0.xh&lcsc_vid=RFZeBFxfRgVYUFRXRFhXUVRVQQJeUAdXQ1FaBAZQEgAxVlNRTlheXldWQlFYVzsOAxUeFF5JWBYZEEoKFBINSQcJGk4dAgUUFAk%3D"
 			(at 106.68 97.79 0)
 			(hide yes)
@@
 			)
 		)
-		(property "Description" "Unpolarized capacitor"
+		(property "Description" "CAP CER 0.8pF 50V C0G 0402"
 			(at 106.68 97.79 0)
 			(hide yes)
@@
 			)
 		)
-		(property "Manufacturer Part Number" "GRM1555C1HR80BA01D"
+		(property "Distributor" "LCSC"
+			(at 106.68 97.79 0)
+			(hide yes)
+			(show_name no)
+			(do_not_autoplace no)
+			(effects
+				(font
+					(size 1.27 1.27)
+				)
+			)
+		)
+		(property "MPN" "GRM1555C1HR80BA01D"
 			(at 106.68 97.79 0)
 			(hide yes)
@@
 			)
 		)
-		(property "Footprint" ""
+		(property "Footprint" "Capacitor_SMD:C_0402_1005Metric"
 			(at 125.4252 101.6 0)
 			(hide yes)
@@
 			)
 		)
-		(property "Datasheet" ""
+		(property "Datasheet" "https://www.lcsc.com/datasheet/C92338.pdf?spm=wm.sxq.inf.ggs___wm.fly.bg.0.xh&lcsc_vid=RFZeBFxfRgVYUFRXRFhXUVRVQQJeUAdXQ1FaBAZQEgAxVlNRTlheXldQT1JbVDsOAxUeFF5JWBYZEEoKFBINSQcJGk4dAgUUFAk%3D"
 			(at 124.46 97.79 0)
 			(hide yes)
@@
 			)
 		)
-		(property "Description" "Unpolarized capacitor"
+		(property "Description" "CAP CER 0.3pF 50V C0G 0402"
 			(at 124.46 97.79 0)
 			(hide yes)
@@
 			)
 		)
-		(property "Manufacturer Part Number" "GRM1555C1HR30WA01D"
+		(property "Distributor" "LCSC"
+			(at 124.46 97.79 0)
+			(hide yes)
+			(show_name no)
+			(do_not_autoplace no)
+			(effects
+				(font
+					(size 1.27 1.27)
+				)
+			)
+		)
+		(property "MPN" "GRM1555C1HR30WA01D"
 			(at 124.46 97.79 0)
 			(hide yes)
@@
 			)
 		)
-		(property "Footprint" ""
+		(property "Footprint" "Inductor_SMD:L_0402_1005Metric"
 			(at 115.57 93.98 0)
 			(hide yes)
@@
 			)
 		)
-		(property "Datasheet" ""
+		(property "Datasheet" "https://www.lcsc.com/datasheet/C77108.pdf?spm=wm.sxq.inf.ggs___wm.fly.bg.0.xh&lcsc_vid=RFZeBFxfRgVYUFRXRFhXUVRVQQJeUAdXQ1FaBAZQEgAxVlNRTlheXlBXRFFfVjsOAxUeFF5JWBYZEEoKFBINSQcJGk4dAgUUFAk%3D"
 			(at 115.57 93.98 0)
 			(hide yes)
@@
 			)
 		)
-		(property "Description" "Inductor"
+		(property "Description" "FIXED IND 2.7nH 800mA 120mΩ 0402"
 			(at 115.57 93.98 0)
 			(hide yes)
@@
 			)
 		)
-		(property "Manufacturer Part Number" "LQG15HS2N7S02D"
+		(property "Distributor" "LCSC"
+			(at 115.57 93.98 90)
+			(hide yes)
+			(show_name no)
+			(do_not_autoplace no)
+			(effects
+				(font
+					(size 1.27 1.27)
+				)
+			)
+		)
+		(property "MPN" "LQG15HS2N7S02D"
 			(at 115.57 93.98 90)
 			(hide yes)
@@
 			)
 		)
-		(property "Manufacturer Part Number" ""
+		(property "Distributor" ""
 			(at 180.34 93.98 0)
 			(hide yes)

Commit message: fix(footprints and symbols): add missing footprints and symbols
Parts:
- removed FL1: TDK_DLF162500LT-5028A1, #odaij_RF_Filter:TDK_DLF162500LT-5028A1, symbol #odaij_RF_Filter:TDK_DLF162500LT-5028A1
- removed J1: Conn_Coaxial, symbol Connector:Conn_Coaxial
- added FL1: DLF162500LT-5028A1, #odaij_RF_Filter:TDK_DLF162500LT-5028A1, symbol #stm32-bt-board-external-symbols:DLF162500LT-5028A1
- added J1: 1909763-1, #stm32-bt-board-external-footprints:1909763-1, symbol #stm32-bt-board-external-symbols:1909763-1
Connections:
- net GND: now also FL1.2 (GND), FL1.4 (GND), J1.2 (Ext), J1.3 (Ext)
- net RF_ANT: now also FL1.3 (OUT), J1.1 (In)
- net RF_MATCH: now also FL1.1 (IN)
Changed lines of the file:
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@@
 		(color 0 0 0 0)
 	)
+	(junction
+		(at 180.34 102.87)
+		(diameter 0)
+		(color 0 0 0 0)
+	)
 	(wire
 		(pts
@@
 	(wire
 		(pts
+			(xy 180.34 102.87) (xy 195.58 102.87)
+		)
+		(stroke
+			(width 0)
+			(type default)
+		)
+	)
+	(wire
+		(pts
+			(xy 195.58 86.36) (xy 180.34 86.36)
+		)
+		(stroke
+			(width 0)
+			(type default)
+		)
+	)
+	(wire
+		(pts
+			(xy 180.34 102.87) (xy 180.34 107.95)
+		)
+		(stroke
+			(width 0)
+			(type default)
+		)
+	)
+	(wire
+		(pts
 			(xy 153.67 100.33) (xy 153.67 104.14)
 		)
@@
 	(wire
 		(pts
-			(xy 180.34 99.06) (xy 180.34 107.95)
+			(xy 180.34 99.06) (xy 180.34 102.87)
+		)
+		(stroke
+			(width 0)
+			(type default)
+		)
+	)
+	(wire
+		(pts
+			(xy 195.58 102.87) (xy 195.58 86.36)
 		)
 		(stroke
@@
 		(pts
 			(xy 124.46 101.6) (xy 124.46 107.95)
+		)
+		(stroke
+			(width 0)
+			(type default)
+		)
+	)
+	(wire
+		(pts
+			(xy 180.34 86.36) (xy 180.34 88.9)
 		)
 		(stroke
@@
 	)
 	(symbol
-		(lib_id "#odaij_RF_Filter:TDK_DLF162500LT-5028A1")
+		(lib_id "#stm32-bt-board-external-symbols:DLF162500LT-5028A1")
 		(at 154.94 93.98 0)
 		(unit 1)
@@
 			)
 		)
-		(property "Value" "TDK_DLF162500LT-5028A1"
+		(property "Value" "DLF162500LT-5028A1"
 			(at 154.94 87.63 0)
 			(show_name no)
@@
 			)
 		)
+		(pin "1"
+		)
+		(pin "3"
+		)
 		(pin "2"
-		)
-		(pin "1"
-		)
-		(pin "3"
 		)
 		(pin "4"
@@
 	)
 	(symbol
+		(lib_id "#stm32-bt-board-external-symbols:1909763-1")
+		(at 180.34 93.98 0)
+		(unit 1)
+		(body_style 1)
+		(exclude_from_sim no)
+		(in_bom yes)
+		(on_board yes)
+		(in_pos_files yes)
+		(dnp no)
+		(fields_autoplaced yes)
+		(property "Reference" "J1"
+			(at 182.88 92.7099 0)
+			(show_name no)
+			(do_not_autoplace no)
+			(effects
+				(font
+					(size 1.27 1.27)
+				)
+				(justify left)
+			)
+		)
+		(property "Value" "1909763-1"
+			(at 182.88 95.2499 0)
+			(show_name no)
+			(do_not_autoplace no)
+			(effects
+				(font
+					(size 1.27 1.27)
+				)
+				(justify left)
+			)
+		)
+		(property "Footprint" "#stm32-bt-board-external-footprints:1909763-1"
+			(at 180.34 93.98 0)
+			(hide yes)
+			(show_name no)
+			(do_not_autoplace no)
+			(effects
+				(font
+					(size 1.27 1.27)
+				)
+			)
+		)
+		(property "Datasheet" "https://www.lcsc.com/datasheet/C392444.pdf?spm=wm.sxq.inf.ggs___wm.fly.bg.0.xh&lcsc_vid=RlRYUFFURFcNVFIDFVMMXgZSRlJeUABSQVNfAwJfQwIxVlNeTllXUVZVRFVXUDsOAxUeFF5JWBYZEEoKFBINSQcJGk4eFQsCAgIaSgADAwAHC0slRlRZXlZQWQkaCgg%3D"
+			(at 180.34 93.98 0)
+			(hide yes)
+			(show_name no)
+			(do_not_autoplace no)
+			(effects
+				(font
+					(size 1.27 1.27)
+				)
+			)
+		)
+		(property "Description" "coaxial connector (BNC, SMA, SMB, SMC, Cinch/RCA, LEMO, ...)"
+			(at 180.34 93.98 0)
+			(hide yes)
+			(show_name no)
+			(do_not_autoplace no)
+			(effects
+				(font
+					(size 1.27 1.27)
+				)
+			)
+		)
+		(property "Distributor" "LCSC"
+			(at 180.34 93.98 0)
+			(hide yes)
+			(show_name no)
+			(do_not_autoplace no)
+			(effects
+				(font
+					(size 1.27 1.27)
+				)
+			)
+		)
+		(pin "3"
+		)
+		(pin "2"
+		)
+		(pin "1"
+		)
+		(instances
+			(project "stm32-bt-board"
+				(path "/9ab97115-0b3b-4897-8d44-f79e27c270d1/647642cc-3894-4f8c-9e36-c4f1abaf1fd9/387be5c2-c06a-4ce1-b441-93a813b84222"
+					(reference "J1")
+					(unit 1)
+				)
+			)
+		)
+	)
+	(symbol
 		(lib_id "Device:C")
 		(at 106.68 97.79 0)
@@
 					(unit 1)
 				)
-			)
-		)
-	)
-	(symbol
-		(lib_id "Connector:Conn_Coaxial")
-		(at 180.34 93.98 0)
-		(unit 1)
-		(body_style 1)
-		(exclude_from_sim no)
-		(in_bom yes)
-		(on_board yes)
-		(in_pos_files yes)
-		(dnp no)
-		(fields_autoplaced yes)
-		(property "Reference" "J1"
-			(at 184.15 93.0031 0)
-			(show_name no)
-			(do_not_autoplace no)
-			(effects
-				(font
-					(size 1.27 1.27)
-				)
-				(justify left)
-			)
-		)
-		(property "Value" "Conn_Coaxial"
-			(at 184.15 95.5431 0)
-			(show_name no)
-			(do_not_autoplace no)
-			(effects
-				(font
-					(size 1.27 1.27)
-				)
-				(justify left)
-			)
-		)
-		(property "Footprint" ""
-			(at 180.34 93.98 0)
-			(hide yes)
-			(show_name no)
-			(do_not_autoplace no)
-			(effects
-				(font
-					(size 1.27 1.27)
-				)
-			)
-		)
-		(property "Datasheet" ""
-			(at 180.34 93.98 0)
-			(hide yes)
-			(show_name no)
-			(do_not_autoplace no)
-			(effects
-				(font
-					(size 1.27 1.27)
-				)
-			)
-		)
-		(property "Description" "coaxial connector (BNC, SMA, SMB, SMC, Cinch/RCA, LEMO, ...)"
-			(at 180.34 93.98 0)
-			(hide yes)
-			(show_name no)
-			(do_not_autoplace no)
-			(effects
-				(font
-					(size 1.27 1.27)
-				)
-			)
-		)
-		(property "KLC_S3.3" ""
-			(at 180.34 93.98 0)
-			(hide yes)
-			(show_name no)
-			(do_not_autoplace no)
-			(effects
-				(font
-					(size 1.27 1.27)
-				)
-			)
-		)
-		(property "KLC_S4.1" ""
-			(at 180.34 93.98 0)
-			(hide yes)
-			(show_name no)
-			(do_not_autoplace no)
-			(effects
-				(font
-					(size 1.27 1.27)
-				)
-			)
-		)
-		(property "Distributor Link" ""
-			(at 180.34 93.98 0)
-			(hide yes)
-			(show_name no)
-			(do_not_autoplace no)
-			(effects
-				(font
-					(size 1.27 1.27)
-				)
-			)
-		)
-		(property "Manufacturer" ""
-			(at 180.34 93.98 0)
-			(hide yes)
-			(show_name no)
-			(do_not_autoplace no)
-			(effects
-				(font
-					(size 1.27 1.27)
-				)
-			)
-		)
-		(property "Distributor" ""
-			(at 180.34 93.98 0)
-			(hide yes)
-			(show_name no)
-			(do_not_autoplace no)
-			(effects
-				(font
-					(size 1.27 1.27)
-				)
-			)
-		)
-		(pin "1"
-		)
-		(pin "2"
-		)
-		(instances
-			(project "stm32-bt-board"
-				(path "/9ab97115-0b3b-4897-8d44-f79e27c270d1/647642cc-3894-4f8c-9e36-c4f1abaf1fd9/387be5c2-c06a-4ce1-b441-93a813b84222"
-					(reference "J1")
-					(unit 1)
-				)

Commit message: fix(symbol): link TDK filter symbol to an existing footprint
Parts:
- FL1: footprint #odaij_RF_Filter:TDK_DLF162500LT-5028A1 -> #stm32-bt-board-external-footprints:DLF162500LT-5028A1
Changed lines of the file:
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@@
 			)
 		)
-		(property "Footprint" "#odaij_RF_Filter:TDK_DLF162500LT-5028A1"
+		(property "Footprint" "#stm32-bt-board-external-footprints:DLF162500LT-5028A1"
 			(at 154.94 93.98 0)
 			(hide yes)

Commit message: i am in a hurry
Other:
- note added: "layout: careful layout needed? answer: yes"
- note removed: "layout: careful layout needed?"
Changed lines of the file:
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@@
 		)
 	)
-	(text "layout: careful layout needed?"
+	(text "layout: careful layout needed?\nanswer: yes"
 		(exclude_from_sim no)
 		(at 101.6 115.062 0)

Commit message: feat(BOM): fill missing parts in BOM
Parts:
- J1: Distributor Link (none) -> https://www.lcsc.com/product-detail/C392444.html?s_z=s_p_19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; MPN (none) -> 1909763-1; Manufacturer (none) -> TE Connectivity
Changed lines of the file:
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@@
 			)
 		)
-		(property "Description" "coaxial connector (BNC, SMA, SMB, SMC, Cinch/RCA, LEMO, ...)"
+		(property "Description" "CONN RCPT IPEX 50Ω SMD"
 			(at 180.34 93.98 0)
 			(hide yes)
@@
 			(at 180.34 93.98 0)
 			(hide yes)
+			(show_name no)
+			(do_not_autoplace no)
+			(effects
+				(font
+					(size 1.27 1.27)
+				)
+			)
+		)
+		(property "Distributor Link" "https://www.lcsc.com/product-detail/C392444.html?s_z=s_p_1909763-1"
+			(at 180.34 93.98 0)
+			(hide yes)
+			(show_name no)
+			(do_not_autoplace no)
+			(effects
+				(font
+					(size 1.27 1.27)
+				)
+			)
+		)
+		(property "MPN" "1909763-1"
+			(at 180.34 93.98 0)
+			(hide yes)
+			(show_name no)
+			(do_not_autoplace no)
+			(effects
+				(font
+					(size 1.27 1.27)
+				)
+			)
+		)
+		(property "Manufacturer" "TE Connectivity"
+			(at 180.34 93.98 0)
+			(hide yes)
