File: kicad/mcu_rf.kicad_sch (KiCad schematic)
At the start: 5 parts, among them J1 1909763-1

Commit message: feat(manuf.): edit BOM and CPL to match JLCPCB's requirements
however, please pay close attention to the rotations during ordering, especially for the SOT components, as JLCPCB messes them up a bit, same for the connector and the filter
Parts:
- C12: Distributor Link https://www.lcsc.com/product-detail/C76988.html?s_z=s_p_GRM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 -> https://www.lcsc.com/product-detail/C76988.html; JLCPCB Part # (none) -> C76988
- C13: Distributor Link https://www.lcsc.com/product-detail/C92338.html?s_z=s_p_GRM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 -> https://www.lcsc.com/product-detail/C92338.html; JLCPCB Part # (none) -> C92338
- FL1: Distributor Link https://www.lcsc.com/product-detail/C531364.html?s_z=s_p_DL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 -> https://www.lcsc.com/product-detail/C531364.html; JLCPCB Part # (none) -> C531364
- J1: Distributor Link https://www.lcsc.com/product-detail/C392444.html?s_z=s_p_19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 -> https://www.lcsc.com/product-detail/C392444.html; JLCPCB Part # (none) -> C392444
- L3: Distributor Link https://www.lcsc.com/product-detail/C77108.html?s_z=s_p_LQG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 -> https://www.lcsc.com/product-detail/C77108.html; JLCPCB Part # (none) -> C77108
Changed lines of the file:
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@@
-			)
-		)
-		(property "Distributor Link" "https://www.lcsc.com/product-detail/C531364.html?s_z=s_p_DLF162500LT-5028A1&spm=wm.fly.bg.0.xh&lcsc_vid=RlRYUFFURFcNVFIDFVMMXgZSRlJeUABSQVNfAwJfQwIxVlNeTldcX1JQQVRbVjsOAxUeFF5JWBYZEEoKFBINSQcJGk4eFQsCAgIaSgADAwAHC0slRVldVVFfWQkaCgg%3D"
-			(at 154.94 93.98 0)
-			(hide yes)
-			(show_name no)
-			(do_not_autoplace no)
-			(effects
-				(font
-					(size 1.27 1.27)
-				)
 			)
 		)
@@
 		)
 		(property "MPN" "DLF162500LT-5028A1"
+			(at 154.94 93.98 0)
+			(hide yes)
+			(show_name no)
+			(do_not_autoplace no)
+			(effects
+				(font
+					(size 1.27 1.27)
+				)
+			)
+		)
+		(property "JLCPCB Part #" "C531364"
+			(at 154.94 93.98 0)
+			(hide yes)
+			(show_name no)
+			(do_not_autoplace no)
+			(effects
+				(font
+					(size 1.27 1.27)
+				)
+			)
+		)
+		(property "Distributor Link" "https://www.lcsc.com/product-detail/C531364.html"
 			(at 154.94 93.98 0)
 			(hide yes)
@@
 			)
 		)
-		(property "Distributor Link" "https://www.lcsc.com/product-detail/C392444.html?s_z=s_p_1909763-1"
-			(at 180.34 93.98 0)
-			(hide yes)
-			(show_name no)
-			(do_not_autoplace no)
-			(effects
-				(font
-					(size 1.27 1.27)
-				)
-			)
-		)
 		(property "MPN" "1909763-1"
 			(at 180.34 93.98 0)
@@
 		)
 		(property "Manufacturer" "TE Connectivity"
+			(at 180.34 93.98 0)
+			(hide yes)
+			(show_name no)
+			(do_not_autoplace no)
+			(effects
+				(font
+					(size 1.27 1.27)
+				)
+			)
+		)
+		(property "JLCPCB Part #" "C392444"
+			(at 180.34 93.98 0)
+			(hide yes)
+			(show_name no)
+			(do_not_autoplace no)
+			(effects
+				(font
+					(size 1.27 1.27)
+				)
+			)
+		)
+		(property "Distributor Link" "https://www.lcsc.com/product-detail/C392444.html"
 			(at 180.34 93.98 0)
 			(hide yes)
@@
 			)
 		)
-		(property "Distributor Link" "https://www.lcsc.com/product-detail/C76988.html?s_z=s_p_GRM1555C1HR80BA01D&spm=wm.fly.bg.0.xh&lcsc_vid=RFZeBFxfRgVYUFRXRFhXUVRVQQJeUAdXQ1FaBAZQEgAxVlNRTlheXldWQlFYVzsOAxUeFF5JWBYZEEoKFBINSQcJGk4dAgUUFAk%3D"
-			(at 106.68 97.79 0)
-			(hide yes)
-			(show_name no)
-			(do_not_autoplace no)
-			(effects
-				(font
-					(size 1.27 1.27)
-				)
-			)
-		)
 		(property "Manufacturer" "muRata"
 			(at 106.68 97.79 0)
@@
 		)
 		(property "MPN" "GRM1555C1HR80BA01D"
+			(at 106.68 97.79 0)
+			(hide yes)
+			(show_name no)
+			(do_not_autoplace no)
+			(effects
+				(font
+					(size 1.27 1.27)
+				)
+			)
+		)
+		(property "JLCPCB Part #" "C76988"
+			(at 106.68 97.79 0)
+			(hide yes)
+			(show_name no)
+			(do_not_autoplace no)
+			(effects
+				(font
+					(size 1.27 1.27)
+				)
+			)
+		)
+		(property "Distributor Link" "https://www.lcsc.com/product-detail/C76988.html"
 			(at 106.68 97.79 0)
 			(hide yes)
@@
 			)
 		)
-		(property "Distributor Link" "https://www.lcsc.com/product-detail/C92338.html?s_z=s_p_GRM1555C1HR30WA01D&spm=wm.fly.bg.0.xh&lcsc_vid=RFZeBFxfRgVYUFRXRFhXUVRVQQJeUAdXQ1FaBAZQEgAxVlNRTlheXldQT1JbVDsOAxUeFF5JWBYZEEoKFBINSQcJGk4dAgUUFAk%3D"
-			(at 124.46 97.79 0)
-			(hide yes)
-			(show_name no)
-			(do_not_autoplace no)
-			(effects
-				(font
-					(size 1.27 1.27)
-				)
-			)
-		)
 		(property "Manufacturer" "muRata"
 			(at 124.46 97.79 0)
@@
 		)
 		(property "MPN" "GRM1555C1HR30WA01D"
+			(at 124.46 97.79 0)
+			(hide yes)
+			(show_name no)
+			(do_not_autoplace no)
+			(effects
+				(font
+					(size 1.27 1.27)
+				)
+			)
+		)
+		(property "JLCPCB Part #" "C92338"
+			(at 124.46 97.79 0)
+			(hide yes)
+			(show_name no)
+			(do_not_autoplace no)
+			(effects
+				(font
+					(size 1.27 1.27)
+				)
+			)
+		)
+		(property "Distributor Link" "https://www.lcsc.com/product-detail/C92338.html"
 			(at 124.46 97.79 0)
 			(hide yes)
@@
 			)
 		)
-		(property "Distributor Link" "https://www.lcsc.com/product-detail/C77108.html?s_z=s_p_LQG15HS2N7S02D&spm=wm.fly.bg.0.xh&lcsc_vid=RFZeBFxfRgVYUFRXRFhXUVRVQQJeUAdXQ1FaBAZQEgAxVlNRTlheXlBXRFFfVjsOAxUeFF5JWBYZEEoKFBINSQcJGk4dAgUUFAk%3D"
-			(at 115.57 93.98 90)
-			(hide yes)
-			(show_name no)
-			(do_not_autoplace no)
-			(effects
-				(font
-					(size 1.27 1.27)
-				)
-			)
-		)
 		(property "Manufacturer" "muRata"
 			(at 115.57 93.98 90)
@@
 			(at 115.57 93.98 90)
 			(hide yes)
+			(show_name no)
+			(do_not_autoplace no)
+			(effects
+				(font
+					(size 1.27 1.27)
+				)
+			)
+		)
+		(property "JLCPCB Part #" "C77108"
+			(at 115.57 93.98 90)
+			(hide yes)
+			(show_name no)
+			(do_not_autoplace no)
+			(effects
+				(font
+					(size 1.27 1.27)
+				)
+			)
+		)
+		(property "Distributor Link" "https://www.lcsc.com/product-detail/C77108.html"
+			(at 115.57 93.98 90)
+			(hide yes)
