File: kicad/mcu_smps.kicad_sch (KiCad schematic)
At the start: 3 parts

Commit message: everything: select real components, refactor schematic, add a user-led driving circuit, and more
Parts:
- C11: footprint (none) -> Capacitor_SMD:C_0603_1608Metric; Distributor (none) -> LCSC; Distributor Link (none) -> https://www.lcsc.com/product-detail/C307467.html?spm=wm.fly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; MPN (none) -> CL10A475KL8NRNC; Manufacturer (none) -> Samsung Electro-Mechanics
- L1: footprint (none) -> Inductor_SMD:L_0402_1005Metric
- L2: footprint (none) -> Inductor_SMD:L_0805_2012Metric
Other:
- note added: "AN5246 How to use SMPS to improve power efficiency on STM32WB MCUs"
- note removed: "https://www.st.com/resource/en/application_note/an5246-how-to-use-smps-to-improve-power-efficiency-on-stm32wb-mcus-stmicroelectronics.pdf"
Changed lines of the file:
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@@
 		)
 	)
-	(text "https://www.st.com/resource/en/application_note/an5246-how-to-use-smps-to-improve-power-efficiency-on-stm32wb-mcus-stmicroelectronics.pdf"
+	(text "AN5246\nHow to use SMPS to improve power efficiency on STM32WB MCUs"
 		(exclude_from_sim no)
-		(at 133.858 94.996 0)
+		(at 125.095 100.965 0)
 		(effects
 			(font
-				(size 0.254 0.254)
-			)
+				(size 1 1)
+				(thickness 0.125)
+			)
+			(href "https://www.st.com/resource/en/application_note/an5246-how-to-use-smps-to-improve-power-efficiency-on-stm32wb-mcus-stmicroelectronics.pdf")
 		)
 	)
@@
 			)
 		)
-		(property "Footprint" ""
+		(property "Footprint" "Inductor_SMD:L_0402_1005Metric"
 			(at 124.46 93.98 0)
 			(hide yes)
@@
 			)
 		)
-		(property "Manufacturer Part Number" ""
+		(property "Distributor" ""
 			(at 124.46 93.98 90)
 			(hide yes)
@@
 			)
 		)
-		(property "Footprint" ""
+		(property "Footprint" "Capacitor_SMD:C_0603_1608Metric"
 			(at 159.7152 102.87 0)
 			(hide yes)
@@
 			)
 		)
-		(property "Datasheet" ""
-			(at 158.75 99.06 0)
-			(hide yes)
-			(show_name no)
-			(do_not_autoplace no)
-			(effects
-				(font
-					(size 1.27 1.27)
-				)
-			)
-		)
-		(property "Description" "Unpolarized capacitor"
+		(property "Datasheet" "https://www.lcsc.com/datasheet/C307467.pdf?spm=wm.sxq.inf.ggs___wm.fly.bg.5.xh&lcsc_vid=RlRYUFFURFcNVFIDFVMMXgZSRlJeUABSQVNfAwJfQwIxVlNeTldcX1VVRFlfUDsOAxUeFF5JWBYZEEoKFBINSQcJGk4eFQsCAgIaSgADAwAHC0slRlNdUVVXWQkaCgg%3D"
+			(at 158.75 99.06 0)
+			(hide yes)
+			(show_name no)
+			(do_not_autoplace no)
+			(effects
+				(font
+					(size 1.27 1.27)
+				)
+			)
+		)
+		(property "Description" "CAP CER 4.7uF 35V X5R 0603"
 			(at 158.75 99.06 0)
 			(hide yes)
@@
 			)
 		)
-		(property "Distributor Link" ""
-			(at 158.75 99.06 0)
-			(hide yes)
-			(show_name no)
-			(do_not_autoplace no)
-			(effects
-				(font
-					(size 1.27 1.27)
-				)
-			)
-		)
-		(property "Manufacturer" ""
-			(at 158.75 99.06 0)
-			(hide yes)
-			(show_name no)
-			(do_not_autoplace no)
-			(effects
-				(font
-					(size 1.27 1.27)
-				)
-			)
-		)
-		(property "Manufacturer Part Number" ""
+		(property "Distributor Link" "https://www.lcsc.com/product-detail/C307467.html?spm=wm.fly.bg.5.xh&lcsc_vid=RlRYUFFURFcNVFIDFVMMXgZSRlJeUABSQVNfAwJfQwIxVlNeTldcX1VVRFlfUDsOAxUeFF5JWBYZEEoKFBINSQcJGk4eFQsCAgIaSgADAwAHC0slRlNdUVVXWQkaCgg%3D"
+			(at 158.75 99.06 0)
+			(hide yes)
+			(show_name no)
+			(do_not_autoplace no)
+			(effects
+				(font
+					(size 1.27 1.27)
+				)
+			)
+		)
+		(property "Manufacturer" "Samsung Electro-Mechanics"
+			(at 158.75 99.06 0)
+			(hide yes)
+			(show_name no)
+			(do_not_autoplace no)
+			(effects
+				(font
+					(size 1.27 1.27)
+				)
+			)
+		)
+		(property "Distributor" "LCSC"
+			(at 158.75 99.06 0)
+			(hide yes)
+			(show_name no)
+			(do_not_autoplace no)
+			(effects
+				(font
+					(size 1.27 1.27)
+				)
+			)
+		)
+		(property "MPN" "CL10A475KL8NRNC"
 			(at 158.75 99.06 0)
 			(hide yes)
@@
 			)
 		)
-		(property "Footprint" ""
+		(property "Footprint" "Inductor_SMD:L_0805_2012Metric"
 			(at 143.51 93.98 0)
 			(hide yes)
@@
 			)
 		)
-		(property "Manufacturer Part Number" ""
+		(property "Distributor" ""
 			(at 143.51 93.98 90)
 			(hide yes)

Commit message: feat(BOM): fill missing parts in BOM
Parts:
- L1: Distributor (none) -> LCSC; Distributor Link (none) -> https://www.lcsc.com/product-detail/C3911026.html?s_z=s_p_L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; MPN (none) -> LQG15WZ10NJ02D; Manufacturer (none) -> muRata
- L2: Distributor (none) -> LCSC; Distributor Link (none) -> https://www.lcsc.com/product-detail/C162582.html?s_z=n_q_LQ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; MPN (none) -> LQM21FN100M80L; Manufacturer (none) -> muRata
Changed lines of the file:
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@@
 			)
 		)
-		(property "Datasheet" ""
+		(property "Datasheet" "https://www.lcsc.com/datasheet/C3911026.pdf"
 			(at 124.46 93.98 0)
 			(hide yes)
@@
 			)
 		)
-		(property "Description" "Inductor"
+		(property "Description" "FIXED IND 10nH 500mA 190mΩ 0402"
 			(at 124.46 93.98 0)
 			(hide yes)
@@
 			)
 		)
-		(property "Distributor Link" ""
-			(at 124.46 93.98 90)
-			(hide yes)
-			(show_name no)
-			(do_not_autoplace no)
-			(effects
-				(font
-					(size 1.27 1.27)
-				)
-			)
-		)
-		(property "Manufacturer" ""
-			(at 124.46 93.98 90)
-			(hide yes)
-			(show_name no)
-			(do_not_autoplace no)
-			(effects
-				(font
-					(size 1.27 1.27)
-				)
-			)
-		)
-		(property "Distributor" ""
+		(property "Distributor Link" "https://www.lcsc.com/product-detail/C3911026.html?s_z=s_p_LQG15WZ10NJ02D"
+			(at 124.46 93.98 90)
+			(hide yes)
+			(show_name no)
+			(do_not_autoplace no)
+			(effects
+				(font
+					(size 1.27 1.27)
+				)
+			)
+		)
+		(property "Manufacturer" "muRata"
+			(at 124.46 93.98 90)
+			(hide yes)
+			(show_name no)
+			(do_not_autoplace no)
+			(effects
+				(font
+					(size 1.27 1.27)
+				)
+			)
+		)
+		(property "Distributor" "LCSC"
+			(at 124.46 93.98 90)
+			(hide yes)
+			(show_name no)
+			(do_not_autoplace no)
+			(effects
+				(font
+					(size 1.27 1.27)
+				)
+			)
+		)
+		(property "MPN" "LQG15WZ10NJ02D"
 			(at 124.46 93.98 90)
 			(hide yes)
@@
 			)
 		)
-		(property "Datasheet" ""
+		(property "Datasheet" "https://www.lcsc.com/datasheet/C162582.pdf"
 			(at 143.51 93.98 0)
 			(hide yes)
@@
 			)
 		)
-		(property "Description" "Inductor"
+		(property "Description" "FIXED IND 10uH 100mA 390mΩ 0805"
 			(at 143.51 93.98 0)
 			(hide yes)
@@
 			)
 		)
-		(property "Distributor Link" ""
-			(at 143.51 93.98 90)
-			(hide yes)
-			(show_name no)
-			(do_not_autoplace no)
-			(effects
-				(font
-					(size 1.27 1.27)
-				)
-			)
-		)
-		(property "Manufacturer" ""
-			(at 143.51 93.98 90)
-			(hide yes)
-			(show_name no)
-			(do_not_autoplace no)
-			(effects
-				(font
-					(size 1.27 1.27)
-				)
-			)
-		)
-		(property "Distributor" ""
-			(at 143.51 93.98 90)
-			(hide yes)
+		(property "Distributor Link" "https://www.lcsc.com/product-detail/C162582.html?s_z=n_q_LQM21FN100M80"
+			(at 143.51 93.98 90)
+			(hide yes)
+			(show_name no)
+			(do_not_autoplace no)
+			(effects
+				(font
+					(size 1.27 1.27)
+				)
+			)
+		)
+		(property "Manufacturer" "muRata"
+			(at 143.51 93.98 90)
+			(hide yes)
+			(show_name no)
+			(do_not_autoplace no)
+			(effects
+				(font
+					(size 1.27 1.27)
+				)
+			)
+		)
+		(property "Distributor" "LCSC"
+			(at 143.51 93.98 90)
+			(hide yes)
+			(show_name no)
+			(do_not_autoplace no)
+			(effects
+				(font
+					(size 1.27 1.27)
+				)
+			)
+		)
+		(property "MPN" "LQM21FN100M80L"
+			(at 143.51 93.98 90)
+			(hide yes)

Commit message: feat(manuf.): edit BOM and CPL to match JLCPCB's requirements
however, please pay close attention to the rotations during ordering, especially for the SOT components, as JLCPCB messes them up a bit, same for the connector and the filter
Parts:
- C11: Distributor Link https://www.lcsc.com/product-detail/C307467.html?spm=wm.fly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 -> https://www.lcsc.com/product-detail/C307467.html; JLCPCB Part # (none) -> C307467
- L1: Distributor Link https://www.lcsc.com/product-detail/C3911026.html?s_z=s_p_L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 -> https://www.lcsc.com/product-detail/C3911026.html; JLCPCB Part # (none) -> C3911026
- L2: Distributor Link https://www.lcsc.com/product-detail/C162582.html?s_z=n_q_LQ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 -> https://www.lcsc.com/product-detail/C162582.html; JLCPCB Part # (none) -> C162582
Changed lines of the file:
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@@
-			)
-		)
-		(property "Distributor Link" "https://www.lcsc.com/product-detail/C3911026.html?s_z=s_p_LQG15WZ10NJ02D"
-			(at 124.46 93.98 90)
-			(hide yes)
-			(show_name no)
-			(do_not_autoplace no)
-			(effects
-				(font
-					(size 1.27 1.27)
-				)
 			)
 		)
@@
 		)
 		(property "MPN" "LQG15WZ10NJ02D"
+			(at 124.46 93.98 90)
+			(hide yes)
+			(show_name no)
+			(do_not_autoplace no)
+			(effects
+				(font
+					(size 1.27 1.27)
+				)
+			)
+		)
+		(property "JLCPCB Part #" "C3911026"
+			(at 124.46 93.98 90)
+			(hide yes)
+			(show_name no)
+			(do_not_autoplace no)
+			(effects
+				(font
+					(size 1.27 1.27)
+				)
+			)
+		)
+		(property "Distributor Link" "https://www.lcsc.com/product-detail/C3911026.html"
 			(at 124.46 93.98 90)
 			(hide yes)
@@
 			)
 		)
-		(property "Distributor Link" "https://www.lcsc.com/product-detail/C307467.html?spm=wm.fly.bg.5.xh&lcsc_vid=RlRYUFFURFcNVFIDFVMMXgZSRlJeUABSQVNfAwJfQwIxVlNeTldcX1VVRFlfUDsOAxUeFF5JWBYZEEoKFBINSQcJGk4eFQsCAgIaSgADAwAHC0slRlNdUVVXWQkaCgg%3D"
-			(at 158.75 99.06 0)
-			(hide yes)
-			(show_name no)
-			(do_not_autoplace no)
-			(effects
-				(font
-					(size 1.27 1.27)
-				)
-			)
-		)
 		(property "Manufacturer" "Samsung Electro-Mechanics"
 			(at 158.75 99.06 0)
@@
 		)
 		(property "MPN" "CL10A475KL8NRNC"
+			(at 158.75 99.06 0)
+			(hide yes)
+			(show_name no)
+			(do_not_autoplace no)
+			(effects
+				(font
+					(size 1.27 1.27)
+				)
+			)
+		)
+		(property "JLCPCB Part #" "C307467"
+			(at 158.75 99.06 0)
+			(hide yes)
+			(show_name no)
+			(do_not_autoplace no)
+			(effects
+				(font
+					(size 1.27 1.27)
+				)
+			)
+		)
+		(property "Distributor Link" "https://www.lcsc.com/product-detail/C307467.html"
 			(at 158.75 99.06 0)
 			(hide yes)
@@
 			)
 		)
-		(property "Distributor Link" "https://www.lcsc.com/product-detail/C162582.html?s_z=n_q_LQM21FN100M80"
-			(at 143.51 93.98 90)
-			(hide yes)
-			(show_name no)
-			(do_not_autoplace no)
-			(effects
-				(font
-					(size 1.27 1.27)
-				)
-			)
-		)
 		(property "Manufacturer" "muRata"
 			(at 143.51 93.98 90)
@@
 			(at 143.51 93.98 90)
 			(hide yes)
+			(show_name no)
+			(do_not_autoplace no)
+			(effects
+				(font
+					(size 1.27 1.27)
+				)
+			)
+		)
+		(property "JLCPCB Part #" "C162582"
+			(at 143.51 93.98 90)
+			(hide yes)
+			(show_name no)
+			(do_not_autoplace no)
+			(effects
+				(font
+					(size 1.27 1.27)
+				)
+			)
+		)
+		(property "Distributor Link" "https://www.lcsc.com/product-detail/C162582.html"
+			(at 143.51 93.98 90)
+			(hide yes)
